File: Bluetooth_Board.kicad_pcb (KiCad board)
At the start: 4 copper layers, 81 x 65 mm, 58 parts, among them J1 5V Power Pins, J11 3V3 Power Pins, J12 GPIO_Connector, J13 Power Select Jumpers, J14 Debug_Pins, J16 61302021821, J18 GPIO_Connector, J19 Power Select Jumpers, J2 SMA PCB END LAUNCH JACK ROUND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, J3 User Button Jumper, J5 Power Pins, J6 USB_B_Micro, J7 BOOT0_Jumper, J9 LCD_I2C3_Connector, U1 STM32WB55RGVx, U3 USBLC6-2SC6, Y1 ABM3B-32.000MHZ-10-R30-B1U-T, Y2 Clock_ECS-327MVATX-7-CN-TR

Commit message: Update
Parts:
- removed C1, C17, C18, C6: 4u7, Capacitor_SMD:C_0805_2012Metric_Pad1.18x1.45mm_HandSolder
- removed C10, C11, C14, C15, C16, C3, C5, C8: 100n, Capacitor_SMD:C_0805_2012Metric_Pad1.18x1.45mm_HandSolder
- removed C13: 1u, Capacitor_SMD:C_0805_2012Metric_Pad1.18x1.45mm_HandSolder
- removed C2: 10n, Capacitor_SMD:C_0805_2012Metric_Pad1.18x1.45mm_HandSolder
- removed C4: 1uF, Capacitor_SMD:C_0805_2012Metric_Pad1.18x1.45mm_HandSolder
- removed FB1: FCM1608KF-601T03, Inductor_SMD:L_0603_1608Metric_Pad1.05x0.95mm_HandSolder
- removed J12: GPIO_Connector, Connector_PinHeader_2.54mm:PinHeader_2x11_P2.54mm_Vertical
- removed J18: GPIO_Connector, Connector_PinHeader_2.54mm:PinHeader_2x10_P2.54mm_Vertical
- removed L2: 10u Murata LQM21FN100M70L, Inductor_SMD:L_0805_2012Metric_Pad1.15x1.40mm_HandSolder
- removed L3: 10n Murata LQG15WZ10NJ02D, Inductor_SMD:L_0402_1005Metric_Pad0.77x0.64mm_HandSolder
- removed R1: 10R, Resistor_SMD:R_0805_2012Metric_Pad1.20x1.40mm_HandSolder
- removed U1: STM32WB55RGVx, Package_DFN_QFN:QFN-68-1EP_8x8mm_P0.4mm_EP6.4x6.4mm
- removed U5: ~, Personal_Project:Button_KMR231GLFS
- removed Y1: ABM3B-32.000MHZ-10-R30-B1U-T, Personal_Project:XTAL_ABM3B-32.000MHZ-10-R30-B1U-T
- removed Y2: Clock_ECS-327MVATX-7-CN-TR, Personal_Project:Clock_ECS327MVATX7CNTR
- added BH1: Battery_Holder_1060TR, Personal_Project:Battery_Holder_1060TR, F.Cu at (159.7, 34.2)
- added C19: 10n, Capacitor_SMD:C_0805_2012Metric_Pad1.18x1.45mm_HandSolder, F.Cu at (104.6, 66.2)
- added C20: 100n, Capacitor_SMD:C_0805_2012Metric_Pad1.18x1.45mm_HandSolder, F.Cu at (97.4, 55.9)
- added C21: 100n, Capacitor_SMD:C_0805_2012Metric_Pad1.18x1.45mm_HandSolder, F.Cu at (99.2, 46.4)
- added C22: 100n, Capacitor_SMD:C_0805_2012Metric_Pad1.18x1.45mm_HandSolder, F.Cu at (110.2, 50.5)
- added C23: 4u7, Capacitor_SMD:C_0805_2012Metric_Pad1.18x1.45mm_HandSolder, F.Cu at (54.9, 67.4)
- added C26: 4u7, Capacitor_SMD:C_0805_2012Metric_Pad1.18x1.45mm_HandSolder, F.Cu at (55.4, 40.0)
- added C27: 100n, Capacitor_SMD:C_0805_2012Metric_Pad1.18x1.45mm_HandSolder, F.Cu at (100.0, 42.5)
- added C28: 4u7, Capacitor_SMD:C_0805_2012Metric_Pad1.18x1.45mm_HandSolder, F.Cu at (104.0, 42.5)
- added C29: 100n, Capacitor_SMD:C_0805_2012Metric_Pad1.18x1.45mm_HandSolder, F.Cu at (96.5, 51.9)
- added C30: 100n, Capacitor_SMD:C_0805_2012Metric_Pad1.18x1.45mm_HandSolder, F.Cu at (92.5, 59.4)
- added C31: 4u7, Capacitor_SMD:C_0805_2012Metric_Pad1.18x1.45mm_HandSolder, F.Cu at (106.0, 46.3)
- added C32: 4u7, Capacitor_SMD:C_0805_2012Metric_Pad1.18x1.45mm_HandSolder, F.Cu at (114.6, 48.0)
- added C33: 100n, Capacitor_SMD:C_0805_2012Metric_Pad1.18x1.45mm_HandSolder, F.Cu at (110.3, 53.2)
- added C34: 100n, Capacitor_SMD:C_0805_2012Metric_Pad1.18x1.45mm_HandSolder, F.Cu at (106.1, 59.5)
- added C35: 1u, Capacitor_SMD:C_0805_2012Metric_Pad1.18x1.45mm_HandSolder, F.Cu at (108.2, 60.6)
- added C36: 1uF, Capacitor_SMD:C_0805_2012Metric_Pad1.18x1.45mm_HandSolder, F.Cu at (104.0, 59.4)
- added FB2: FCM1608KF-601T03, Inductor_SMD:L_0603_1608Metric_Pad1.05x0.95mm_HandSolder, F.Cu at (111.0, 59.4)
- added IC1: STM32WB55CGU6, Personal_Project:STM32WB55CGU6_QFN50P700X700X60-49N-D, F.Cu at (104.0, 53.1)
- added J10: LPUART1_Header, Connector_PinHeader_2.54mm:PinHeader_1x04_P2.54mm_Vertical, F.Cu at (112.1, 73.1)
- added J15: USART1_Header, Connector_PinHeader_2.54mm:PinHeader_1x04_P2.54mm_Vertical, F.Cu at (120.4, 68.6)
- added J20: SPI1_Header, Connector_PinHeader_2.54mm:PinHeader_1x06_P2.54mm_Vertical, F.Cu at (97.3, 82.3)
- added J4: Coin Battery Jumper, Connector_PinHeader_2.54mm:PinHeader_1x03_P2.54mm_Vertical, F.Cu at (88.0, 59.0)
- added J8: BOOT0_Jumper, Connector_PinHeader_2.54mm:PinHeader_1x03_P2.54mm_Vertical, F.Cu at (91.6, 63.8)
- added L4: 10u Murata LQM21FN100M70L, Inductor_SMD:L_0805_2012Metric_Pad1.15x1.40mm_HandSolder, F.Cu at (103.8, 46.4)
- added L5: 10n Murata LQG15WZ10NJ02D, Inductor_SMD:L_0402_1005Metric_Pad0.77x0.64mm_HandSolder, F.Cu at (102.1, 47.5)
- added U2: ~, Personal_Project:Button_KMR231GLFS, F.Cu at (59.0, 34.5)
- added Y3: Clock_ECS-327MVATX-7-CN-TR, Personal_Project:Clock_ECS327MVATX7CNTR, F.Cu at (98.3, 66.3)
- added Y4: ABM3B-32.000MHZ-8-R30-B1U-T, Personal_Project:XTAL_ABM3B-32.000MHZ-10-R30-B1U-T, F.Cu at (110.3, 45.7)
- J13: value Power Select Jumpers -> 3V3 Power Source Jumpers
- J16: value 61302021821 -> Pin_Header; footprint Personal_Project:WR-PHD 2.54 MM DUAL SOCKET HEADE -> Connector_PinHeader_2.54mm:PinHeader_2x07_P2.54mm_Vertical
- J17: moved to F.Cu
- J7: value BOOT0_Jumper -> I2C3_Header; footprint Connector_PinHeader_2.54mm:PinHeader_1x03_P2.54mm_Vertical -> Connector_PinHeader_2.54mm:PinHeader_1x04_P2.54mm_Vertical
- J9: value LCD_I2C3_Connector -> I2C1_Header
- R2: value 1k -> 10R
- moved U6 144.0 mm to (179.5, 89.2), turned to 0 degrees
- moved J3 138.3 mm to (174.1, 103.5), turned to 0 degrees
- moved R6 133.1 mm to (180.8, 83.6), turned to 0 degrees
- moved J19 131.4 mm to (182.5, 96.3)
- moved J17 128.3 mm to (2.15, 3.55), turned to 0 degrees
- moved C9 127.8 mm to (159.8, 102.6)
- moved J14 126.5 mm to (176.2, 81.5)
- moved ESD1 126.2 mm to (169.6, 103.0), turned to 0 degrees
- moved ESD2 117.8 mm to (169.6, 106.8), turned to 0 degrees
- moved J13 115.5 mm to (175.3, 96.3)
- moved J5 115.2 mm to (159.7, 81.5)
- moved C24 110.8 mm to (159.8, 105.7), turned to 0 degrees
- moved C25 108.5 mm to (159.8, 108.7), turned to 0 degrees
- moved J1 103.7 mm to (159.7, 93.8)
- moved J11 100.6 mm to (166.9, 93.8)
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Connections:
- J14 pad 2: /SWDIO -> /PA13_SWDIO
- J14 pad 4: /SWCLK -> /PA14_SWCLK
- J14 pad 6: /SWO -> /PB3_SWO
- J16 pad 1: /PC10 -> GND
- J16 pad 10: GND -> /PE4
- J16 pad 11: GND -> /PB1
- J16 pad 12: /PB4 -> /PB0
- J16 pad 13: /PB5 -> /AT1
- J16 pad 14: GND -> /AT0
- J16 pad 2: GND -> /PB2
- J16 pad 3: GND -> /PA8_MCO
- J16 pad 4: /PC11 -> /PA5
- J16 pad 5: /PC12 -> /PA0
- J16 pad 6: GND -> /PC15-OSC32_OUT
- J16 pad 7: GND -> /PB7
- J16 pad 8: /PD0 -> /PB6
- J16 pad 9: /PD1 -> /PA15
- J3 pad 2: /PB8_I2C1_SCL -> /PA0
- J7 pad 2: /BOOT0J -> GND
- J7 pad 3: GND -> /PA7_I2C3_SCL
- J9 pad 1: GND -> +3.3V
- J9 pad 2: +5V -> GND
- J9 pad 3: /PC1_I2C3_SDA -> /PB8_I2C1_SCL
- J9 pad 4: /PC0_I2C3_SCL -> /PB9_I2C1_SDA
- R2 pad 1: /BOOT0J -> Net-(Y3-OUTPUT)
- R2 pad 2: /BOOT0 -> Net-(IC1-PC14-OSC32_IN)
- U3 pad 4: /USB_D+ -> /PA12_USB_D+
- U3 pad 6: /USB_D- -> /PA11_USB_D-
Routing:
- net +3.3V: track 280.1 -> 0.00 mm, vias 5 -> 0
- net /NRST: track 105.6 -> 0.00 mm, vias 5 -> 0
- net /PB8_I2C1_SCL: track 104.7 -> 0.00 mm, vias 3 -> 0
- net /PC13: track 81.1 -> 0.00 mm, vias 2 -> 0
- net /PB5: track 78.6 -> 0.00 mm, vias 2 -> 0
- net /PB4: track 76.0 -> 0.00 mm, vias 2 -> 0
- net /PD1: track 71.8 -> 0.00 mm, vias 2 -> 0
- net /PD0: track 69.4 -> 0.00 mm, vias 2 -> 0
- net /PC12: track 66.1 -> 0.00 mm, vias 2 -> 0
- net /PC11: track 64.5 -> 0.00 mm, vias 2 -> 0
- net /SWDIO: track 59.7 -> 0.00 mm, vias 1 -> 0
- net /SWO: track 58.7 -> 0.00 mm, vias 2 -> 0
- net /PC10: track 58.6 -> 0.00 mm, vias 2 -> 0
- net /SWCLK: track 56.7 -> 0.00 mm, vias 2 -> 0
- net +5V: track 52.9 -> 0.00 mm, vias 2 -> 0
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Other:
- board text removed: "3V3/GND"
- board text removed: "5V/GND"
- board text removed: "A0"
- board text removed: "A1"
- board text removed: "A10"
- board text removed: "A15"
- board text removed: "A2"
- board text removed: "A3"
- board text removed: "A4"
- board text removed: "A5"
- board text removed: "A6"
- board text removed: "A7"
- board text removed: "A8"
- board text removed: "A9"
- board text removed: "B0"
- board text removed: "B1"
- board text removed: "B10"
- board text removed: "B11"
- board text removed: "B12"
- board text removed: "B13"
- board text removed: "B14"
- board text removed: "B15"
- board text removed: "B2"
- board text removed: "B4"
- board text removed: "B5"
- board text removed: "B6"
- board text removed: "B7"
- board text removed: "B8"
- board text removed: "B9"
- board text removed: "C0"
- board text removed: "C1"
- board text removed: "C10"
- board text removed: "C11"
- board text removed: "C12"
- board text removed: "C13"
- board text removed: "C2"
- board text removed: "C3"
- board text removed: "C4"
- board text removed: "C5"
- board text removed: "C6"
- board text removed: "D0"
- board text removed: "D1"
- board text removed: "E4"
- board text removed: "GND"
- board text removed: "RST"
- board text removed: "SW/PC/LD"
- board text removed: "SW/PC/VBUS"
- board text removed: "USRBTN/B8"

Commit message: Update
Parts:
- removed J16: Pin_Header, Connector_PinHeader_2.54mm:PinHeader_2x07_P2.54mm_Vertical
- added J12: Pin_Header, Connector_PinHeader_2.54mm:PinHeader_2x06_P2.54mm_Vertical, F.Cu at (100.0, 29.2)
- C19, C20, C21, C22, C23, C24, C25, C26, C27, C28, C29, C30, C31, C32, C33, C34, C35, C36, C9: footprint Capacitor_SMD:C_0805_2012Metric_Pad1.18x1.45mm_HandSolder -> Capacitor_SMD:C_0603_1608Metric_Pad1.08x0.95mm_HandSolder
- J14: footprint Connector_PinSocket_2.54mm:PinSocket_2x04_P2.54mm_Vertical -> Connector_PinHeader_2.54mm:PinHeader_2x04_P2.54mm_Vertical
- moved J17 137.0 mm to (130.1, 52.6)
- moved J19 120.0 mm to (75.6, 41.7), turned to -90 degrees
- moved R6 118.9 mm to (75.0, 29.4)
- moved ESD1 117.4 mm to (73.0, 36.4), turned to 90 degrees
- moved J14 110.7 mm to (70.0, 50.4)
- moved J3 110.0 mm to (95.5, 26.5)
- moved U6 109.6 mm to (87.7, 29.2)
- moved ESD2 105.5 mm to (75.6, 58.9), turned to 90 degrees
- moved J5 102.4 mm to (68.3, 35.4)
- moved J13 102.0 mm to (77.0, 69.0), turned to -90 degrees
- moved C24 102.0 mm to (77.0, 46.0)
- moved C9 100.6 mm to (90.7, 29.5)
- moved J11 99.0 mm to (70.1, 72.7), turned to 180 degrees
- moved C25 98.0 mm to (77.4, 55.7)
- moved J1 91.8 mm to (82.3, 44.4)
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Connections:
- IC1 pad 26: /AT0 -> unconnected-(IC1-AT0-Pad26)
- IC1 pad 27: /AT1 -> unconnected-(IC1-AT1-Pad27)

Commit message: Update
Parts:
- moved C32 4.06 mm to (110.8, 49.9), turned to 90 degrees
- moved C28 1.55 mm to (100.2, 44.6)
- moved C22 1.39 mm to (109.1, 49.9), turned to 90 degrees
- moved Y4 1.20 mm to (110.4, 44.5)
- moved C27 1.03 mm to (100.2, 46.3)
- moved FLT1 0.69 mm to (118.0, 51.9)
- moved C12 0.68 mm to (112.6, 52.5)
- moved C7 0.68 mm to (116.1, 52.5)
- moved L1 0.68 mm to (114.4, 51.9)
- moved J2 0.67 mm to (121.4, 51.9)
- moved C21 0.55 mm to (100.2, 48.0)
- moved C31 0.36 mm to (104.8, 42.6)
- moved C33 0.19 mm to (110.4, 53.0)
Routing:
- net +3.3V: track 0.00 -> 13.3 mm
- net /OSC_IN: track 0.00 -> 8.61 mm
- net GND: track 0.00 -> 7.94 mm
- net /OSC_OUT: track 0.00 -> 7.27 mm
- net /SMPS_FB: track 0.00 -> 6.71 mm
- net /RF1: track 0.00 -> 6.35 mm
- net /RF_ANT: track 0.00 -> 2.73 mm
- net /RF_MATCH: track 0.00 -> 2.42 mm
- net /SMPS_LXL: track 0.00 -> 1.74 mm
- net /SMPS_LX: track 0.00 -> 1.53 mm

Commit message: Update
Parts:
- removed J12: Pin_Header, Connector_PinHeader_2.54mm:PinHeader_2x06_P2.54mm_Vertical
- C22, C32, C33: moved to B.Cu
- J7: value I2C3_Header -> Pin_Header; footprint Connector_PinHeader_2.54mm:PinHeader_1x04_P2.54mm_Vertical -> Connector_PinHeader_2.54mm:PinHeader_2x07_P2.54mm_Vertical
- R2, R6: footprint Resistor_SMD:R_0805_2012Metric_Pad1.20x1.40mm_HandSolder -> Resistor_SMD:R_0603_1608Metric_Pad0.98x0.95mm_HandSolder
- moved J15 50.6 mm to (70.2, 75.1), turned to 90 degrees
- moved J7 49.4 mm to (98.3, 29.9), turned to 90 degrees
- moved H5 33.9 mm to (59.8, 16.8)
- moved J10 28.4 mm to (85.0, 81.7)
- moved J14 21.3 mm to (48.7, 50.4)
- moved C23 19.0 mm to (58.2, 49.1)
- moved C26 19.0 mm to (58.3, 73.5)
- moved C36 19.0 mm to (54.4, 63.1)
- moved J1 19.0 mm to (63.4, 44.5)
- moved J19 19.0 mm to (56.6, 41.8)
- moved LDO1 19.0 mm to (56.2, 52.5)
- moved C25 19.0 mm to (58.4, 55.8)
- moved ESD1 19.0 mm to (54.0, 36.5)
- moved J13 19.0 mm to (58.0, 69.1)
- moved J5 19.0 mm to (49.3, 35.5)
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Connections:
- IC1 pad 10: /PA1_SPI1_SCK -> /PA1
- IC1 pad 14: /PA5 -> /PA5_SPI1_SCK
- IC1 pad 16: /PA7_I2C3_SCL -> /PA7_SPI1_MOSI
- IC1 pad 18: /PA9_USART1_TX -> /PA9
- IC1 pad 3: /PC15-OSC32_OUT -> unconnected-(IC1-PC15-OSC32_OUT-Pad3)
- IC1 pad 36: /PA10_USART1_RX -> /PA10
- IC1 pad 44: /PB4_I2C3_SDA -> /PB4
- IC1 pad 45: /PB5_SPI1_MOSI -> /PB5
- IC1 pad 46: /PB6 -> /PB6_USART1_TX
- IC1 pad 47: /PB7 -> /PB7_USART1_RX
- J15 pad 3: /PA9_USART1_TX -> /PB6_USART1_TX
- J15 pad 4: /PA10_USART1_RX -> /PB7_USART1_RX
- J20 pad 3: /PA1_SPI1_SCK -> /PA7_SPI1_MOSI
- J20 pad 5: /PB5_SPI1_MOSI -> /PA5_SPI1_SCK
- J7 pad 1: +3.3V -> /PB2
- J7 pad 3: /PA7_I2C3_SCL -> /PA8_MCO
- J7 pad 4: /PB4_I2C3_SDA -> /PA9
Routing:
- net +3.3V: track 13.3 -> 193.1 mm, vias 0 -> 7
- net /PB2: track 0.00 -> 79.0 mm, vias 0 -> 2
- net /PA9: track 0.00 -> 76.9 mm, vias 0 -> 2
- net /PA8_MCO: track 0.00 -> 68.4 mm, vias 0 -> 2
- net /PA1: track 0.00 -> 61.5 mm, vias 0 -> 2
- net /PA0: track 0.00 -> 57.7 mm, vias 0 -> 2
- net /NRST: track 0.00 -> 55.3 mm, vias 0 -> 3
- net /PB8_I2C1_SCL: track 0.00 -> 44.2 mm, vias 0 -> 1
- net /PB9_I2C1_SDA: track 0.00 -> 42.9 mm, vias 0 -> 1
- net /PA2_LPUART1_TX: track 0.00 -> 41.1 mm, vias 0 -> 1
- net /PA3_LPUART1_RX: track 0.00 -> 39.9 mm, vias 0 -> 1
- net /PA4_SPI1_NSS: track 0.00 -> 36.9 mm, vias 0 -> 1
- net /PA5_SPI1_SCK: track 0.00 -> 36.5 mm, vias 0 -> 1
- net /PA7_SPI1_MOSI: track 0.00 -> 36.1 mm, vias 0 -> 1
- net /PA6_SPI1_MISO: track 0.00 -> 36.0 mm, vias 0 -> 1
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Other:
- board text added: "B10"
- board text added: "BOOT0 UPD/STR"
- board text added: "VBAT VDD/BAT"

Commit message: Update
Parts:
- moved C24 19.6 mm to (76.9, 40.8), turned to 90 degrees
- moved J13 17.2 mm to (75.2, 69.7)
- moved J1 16.8 mm to (79.9, 41.7)
- moved LDO1 16.3 mm to (72.5, 51.5)
- moved ESD2 16.1 mm to (72.8, 58.6)
- moved H1 16.0 mm to (64.0, 27.0)
- moved H4 16.0 mm to (64.0, 82.0)
- moved ESD1 16.0 mm to (69.9, 34.9)
- moved C25 15.9 mm to (74.3, 55.0)
- moved J11 15.7 mm to (66.8, 73.6)
- moved J14 15.7 mm to (64.3, 48.7)
- moved U2 15.4 mm to (63.0, 63.8)
- moved C36 15.4 mm to (69.8, 62.2)
- moved J5 15.0 mm to (64.3, 34.0)
- moved J19 14.8 mm to (71.3, 40.3)
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Connections:
- ESD1 pad 1: unconnected-(ESD1-I/O1-Pad1) -> /5V_SW
- ESD1 pad 3: /5V_SW -> unconnected-(ESD1-I/O2-Pad3)
- J7 pad 8: /PC15-OSC32_OUT -> GND
Routing:
- net /5V_SW: track 0.00 -> 21.4 mm
- net /VBUS: track 0.00 -> 15.5 mm
- net /PC_5V: track 0.00 -> 15.0 mm
Other:
- board size 81 x 65 mm -> 65 x 65 mm

Commit message: Update
Parts:
- BH1, C29: moved to B.Cu
- moved BH1 56.9 mm to (147.6, 62.3), turned to 180 degrees
- moved H6 43.5 mm to (83.6, 48.4)
- moved H5 37.6 mm to (92.2, 35.8)
- moved C23 8.13 mm to (76.9, 40.8), turned to 90 degrees
- moved LDO1 5.80 mm to (77.2, 48.1)
- moved C25 4.88 mm to (77.3, 51.1), turned to 180 degrees
- moved C24 4.79 mm to (79.0, 45.1), turned to 0 degrees
- moved ESD2 2.26 mm to (75.0, 58.4)
- moved C29 1.52 mm to (95.9, 54.8), turned to -90 degrees
- moved U6 0.87 mm to (85.0, 29.2)
- moved J9 0.80 mm to (71.6, 81.7)
- moved R6 0.67 mm to (72.0, 28.5)
- moved J6 0.56 mm to (75.7, 25.1)
- moved C9 0.55 mm to (88.6, 30.5)
- moved C36 0.22 mm to (69.6, 62.3)
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Connections:
- net /PA11_USB_D- renamed /USB_D-
- net /PA12_USB_D+ renamed /USB_D+
- ESD2 pad 1: unconnected-(ESD2-I/O1-Pad1) -> /3V3_SW
- ESD2 pad 3: /3V3_SW -> unconnected-(ESD2-I/O2-Pad3)
Routing:
- net /PC_3V3: track 0.00 -> 43.0 mm, vias 0 -> 1
- net /USB_D+: track 0.00 -> 38.3 mm
- net /USB_D-: track 0.00 -> 38.2 mm
- net /PA14_SWCLK: track 0.00 -> 34.0 mm, vias 0 -> 1
- net /PA13_SWDIO: track 0.00 -> 33.9 mm, vias 0 -> 1
- net /PB3_SWO: track 0.00 -> 32.6 mm, vias 0 -> 1
- net +5V: track 0.00 -> 25.6 mm
- net /PB4: track 0.00 -> 24.7 mm, vias 0 -> 1
- net /3V3_SW: track 0.00 -> 23.3 mm, vias 0 -> 1
- net +3.3V: track 192.7 -> 215.3 mm, vias 7 -> 8
- net /PB5: track 0.00 -> 22.1 mm, vias 0 -> 1
- net /PA15: track 0.00 -> 22.0 mm, vias 0 -> 1
- net /LD_OUT_3V3: track 0.00 -> 21.0 mm
- net /NRST: track 55.3 -> 71.0 mm, vias 3 -> 4
- net /VBUS: track 15.5 -> 27.3 mm, vias 0 -> 3
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Other:
- board text added: "3V/GN/CL/DA"
- board text added: "3V/GN/TX/RX"
- board text added: "3V3"
- board text added: "5V"
- board text added: "GND"
- board text added: "GND/3V3"
- board text added: "I2C1"
- board text added: "LU1"
- board text added: "NRST"
- board text added: "NS/CK/MI/MO/GN/3V"
- board text added: "SPI1"
- board text added: "SWCLK"
- board text added: "SWIO"
- board text added: "SWO"
- board text added: "USR BTN"
- board text added: "UT1"

Commit message: Update
Parts:
- removed H5: MountingHole_Pad, MountingHole:MountingHole_3.2mm_M3_Pad
- J10: footprint Connector_PinHeader_2.54mm:PinHeader_1x04_P2.54mm_Vertical -> Connector_PinHeader_2.54mm:PinHeader_1x04_P2.54mm_Horizontal
- J20: footprint Connector_PinHeader_2.54mm:PinHeader_1x06_P2.54mm_Vertical -> Connector_PinHeader_2.54mm:PinHeader_1x06_P2.54mm_Horizontal
- moved BH1 48.0 mm to (105.4, 39.6), turned to 0 degrees
- moved J10 7.68 mm to (92.7, 81.7), turned to -90 degrees
- moved H6 0.36 mm to (83.8, 48.7)
- moved J3 0.11 mm to (92.7, 27.3)
Connections:
- J10 pad 1: +3.3V -> /PA3_LPUART1_RX
- J10 pad 2: GND -> /PA2_LPUART1_TX
- J10 pad 3: /PA2_LPUART1_TX -> GND
- J10 pad 4: /PA3_LPUART1_RX -> +3.3V
- J7 pad 1: /PB2 -> /PA1
- J7 pad 3: /PA8_MCO -> /PB2
- J7 pad 4: /PA9 -> /PA0
- J7 pad 5: /PA0 -> /PA8_MCO
- J7 pad 6: /PA1 -> /PA9
Routing:
- net /PA0: track 54.8 -> 100.6 mm, vias 2 -> 3
- net /PA9: track 74.0 -> 119.3 mm, vias 2 -> 3
- net /PA1: track 57.9 -> 100.8 mm, vias 2 -> 3
- net /PB2: track 77.0 -> 119.5 mm, vias 2 -> 3
- net /PA8_MCO: track 68.4 -> 110.4 mm, vias 2 -> 5
- net /PA10: track 0.00 -> 36.4 mm, vias 0 -> 1
- net /PB6_USART1_TX: track 7.31 -> 37.8 mm, vias 0 -> 1
- net /PB7_USART1_RX: track 7.25 -> 34.4 mm, vias 0 -> 1
- net /PB5: track 22.1 -> 46.1 mm, vias 1 -> 3
- net /PB4: track 24.7 -> 47.5 mm, vias 1 -> 3
- net /PA15: track 22.0 -> 38.3 mm, vias 1 -> 3
- net Net-(BH1-+): track 0.00 -> 11.2 mm
- net +3.3V: track 215.3 -> 213.7 mm
- net /PA2_LPUART1_TX: track 41.1 -> 41.7 mm
- net /PA3_LPUART1_RX: track 39.9 -> 40.4 mm
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Other:
- board text added: "5V/GN"
- board text added: "SW/PC/VB"

Commit message: Update
Connections:
- J3 pad 2: /PA0 -> /PA1
Routing:
- net Net-(BH1-+): track 11.2 -> 36.4 mm, vias 0 -> 2
- net Net-(J3-Pin_1): track 0.00 -> 6.78 mm
- net /PA1: track 100.8 -> 106.4 mm
- net GND: vias 77 -> 104
