File: Bluetooth_Board.kicad_pcb (KiCad board)
At the start: 4 copper layers, 100 x 50 mm, 69 parts, among them IC1 STM32WB55CGU6, J1 USART1_Headers, J10 Debug_Pins, J12 Power_Selector_Jumper, J13 General_Pin_Header, J14 JST_XH_2.54_Plug, J15 LPUART1_Headers, J16 SPI1_Headers, J19 3V_Selection_Header, J2 SMA PCB END LAUNCH JACK ROUND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, J3 User Button Jumper, J4 Coin Battery Jumper, J5 USB_B_Micro, J6 I2C1_Headers, J7 General_Pin_Header, J8 BOOT0_Jumper, Q1 MOSFET_SI2333DDS-T1-BE3, U3 USBLC6-2SC6, Y4 ABM3B-32.000MHZ-8-R30-B1U-T

Commit message: Update
Parts:
- removed BH1: Battery_Holder_1060TR, Personal_Project:Battery_Holder_1060TR
- removed C22, C29, C30, C33, C34: 100n, Capacitor_SMD:C_0805_2012Metric
- removed C24, C25, C35: 1u, Capacitor_SMD:C_0805_2012Metric
- removed C31, C32: 4u7, Capacitor_SMD:C_0805_2012Metric
- removed C36: 1uF, Capacitor_SMD:C_0805_2012Metric
- removed D2: BZX84C6V2LT1G, Package_TO_SOT_SMD:SOT-23
- removed IC1: STM32WB55CGU6, Personal_Project:STM32WB55CGU6_QFN50P700X700X60-49N-D
- removed J1: USART1_Headers, Connector_PinHeader_2.54mm:PinHeader_2x03_P2.54mm_Horizontal
- removed J10: Debug_Pins, Connector_PinHeader_2.54mm:PinHeader_2x04_P2.54mm_Horizontal
- removed J12: Power_Selector_Jumper, Connector_PinHeader_2.54mm:PinHeader_2x03_P2.54mm_Vertical
- removed J13: General_Pin_Header, Connector_PinHeader_2.54mm:PinHeader_2x07_P2.54mm_Horizontal
- removed J14: JST_XH_2.54_Plug, Personal_Project:Connector_Power2pin_SHDRRA2W80P0X250_1X2_740X1150X610P
- removed J15: LPUART1_Headers, Connector_PinHeader_2.54mm:PinHeader_2x03_P2.54mm_Horizontal
- removed J16: SPI1_Headers, Connector_PinHeader_2.54mm:PinHeader_2x03_P2.54mm_Horizontal
- removed J19: 3V_Selection_Header, Connector_PinHeader_2.54mm:PinHeader_1x03_P2.54mm_Vertical
- removed J8: BOOT0_Jumper, Connector_PinHeader_2.54mm:PinHeader_1x03_P2.54mm_Vertical
- removed L4: 10u Murata LQM21FN100M70L, Inductor_SMD:L_0805_2012Metric_Pad1.15x1.40mm_HandSolder
- removed L5: 10n Murata LQG15WZ10NJ02D, Inductor_SMD:L_0402_1005Metric_Pad0.77x0.64mm_HandSolder
- removed OS2: Oscillator_ECS-327MVATX-3-CN-TR, Personal_Project:Oscillator_ECS327MVATX3CNTR
- removed R1, R11, R12, R13, R14: 33R, Resistor_SMD:R_0805_2012Metric
- removed R2: 10R, Resistor_SMD:R_0805_2012Metric
- removed R20: 100k, Resistor_SMD:R_0805_2012Metric
- removed S2: Switch_WS-SLSU SMT Mini Slide, Personal_Project:Switch_WS-SLSU SMT Mini Slide
- removed U3: USBLC6-2SC6, Package_TO_SOT_SMD:SOT-23-6
- removed U6: ~, Personal_Project:Button_KMR231GLFS
- removed Y4: ABM3B-32.000MHZ-8-R30-B1U-T, Personal_Project:XTAL_ABM3B-32.000MHZ-10-R30-B1U-T
- removed Z1: Diode_BZX84C6V2-7-F, Personal_Project:Diode_BZX84C6V2_SOT96P240X110-3N
- added BH2: Battery_Holder_1060TR, Personal_Project:Battery_Holder_1060TR, B.Cu at (142.5, 96.5)
- added C1: 4u7, Capacitor_SMD:C_0805_2012Metric, F.Cu at (180.0, 81.7)
- added C10: 100n, Capacitor_SMD:C_0805_2012Metric, F.Cu at (186.7, 99.7)
- added C11: 100n, Capacitor_SMD:C_0805_2012Metric, F.Cu at (170.9, 94.5)
- added C13: 100n, Capacitor_SMD:C_0805_2012Metric, F.Cu at (171.2, 100.9)
- added C14: 100n, Capacitor_SMD:C_0805_2012Metric, F.Cu at (174.3, 101.6)
- added C15: 100n, Capacitor_SMD:C_0805_2012Metric, F.Cu at (133.5, 100.5)
- added C16: 10n, Capacitor_SMD:C_0805_2012Metric, F.Cu at (173.6, 109.8)
- added C18: 4u7, Capacitor_SMD:C_0805_2012Metric, F.Cu at (139.9, 100.6)
- added C26: 100n, Capacitor_SMD:C_0805_2012Metric, F.Cu at (107.2, 90.9)
- added C3: 100n, Capacitor_SMD:C_0805_2012Metric, F.Cu at (170.9, 89.7)
- added C4: 4u7, Capacitor_SMD:C_0805_2012Metric, F.Cu at (175.0, 84.8)
- added C5: 100n, Capacitor_SMD:C_0805_2012Metric, F.Cu at (175.1, 87.2)
- added C6: 4u7, Capacitor_SMD:C_0805_2012Metric, F.Cu at (189.6, 90.0)
- added C8: 100n, Capacitor_SMD:C_0805_2012Metric, F.Cu at (187.2, 90.0)
- added FB2: BLM21AG121BH1D, Capacitor_SMD:C_0805_2012Metric, F.Cu at (136.7, 99.6)
- added FPC1: FPC_0545481072, Personal_Project:FPC_0545481072, F.Cu at (167.3, 116.2)
- added FPC2: FPC_0545482072, Personal_Project:FPC_0545482072, F.Cu at (183.0, 116.0)
- added IC2: STM32WB55CGU6, Personal_Project:STM32WB55CGU6_QFN50P700X700X60-49N-D, F.Cu at (179.2, 95.8)
- added J11: BOOT0_Jumper, Connector_PinHeader_2.54mm:PinHeader_1x03_P2.54mm_Vertical, F.Cu at (164.5, 90.7)
- added J18: User Button Jumper, Connector_PinHeader_2.54mm:PinHeader_1x02_P2.54mm_Vertical, F.Cu at (219.6, 85.3)
- added J24: SWDB, Connector_PinHeader_2.54mm:PinHeader_2x04_P2.54mm_Horizontal, F.Cu at (107.5, 87.9)
- added J9: Coin Battery Jumper, Connector_PinHeader_2.54mm:PinHeader_1x03_P2.54mm_Vertical, F.Cu at (164.4, 102.4)
- added JST1: JST_S3B-XH-2.54, Personal_Project:JST_S3B-XH-SHDRRA3W64P0X250_1X3_990X1150X610P, F.Cu at (118.0, 78.5)
- added L2: 10u Murata LQM21FN100M70L, Inductor_SMD:L_0805_2012Metric_Pad1.15x1.40mm_HandSolder, F.Cu at (179.1, 84.8)
- added L3: 10n Murata LQG15WZ10NJ02D, Inductor_SMD:L_0805_2012Metric_Pad1.05x1.20mm_HandSolder, F.Cu at (178.1, 88.0)
- added OS1: Oscillator_ECS-327MVATX-3-CN-TR, Personal_Project:Oscillator_ECS327MVATX3CNTR, F.Cu at (173.4, 106.5)
- added R4: 10R, Resistor_SMD:R_0805_2012Metric, F.Cu at (176.9, 104.5)
- added R5: 33R, Resistor_SMD:R_0805_2012Metric, F.Cu at (146.1, 82.0)
- added R7: 5k1, Resistor_SMD:R_0805_2012Metric, F.Cu at (113.4, 102.5)
- added R8: 5k1, Resistor_SMD:R_0805_2012Metric, F.Cu at (113.5, 108.8)
- added U4: SN74LVC1G07DBVR, Package_TO_SOT_SMD:SOT-23-5, F.Cu at (134.3, 88.4)
- added U5: USBLC6-2SC6, Package_TO_SOT_SMD:SOT-23-6, F.Cu at (113.8, 105.6)
- added VS1: VS_STM1818TWX7F, Personal_Project:SOT-23-3_SOT103P237X112-3N, F.Cu at (134.4, 96.5)
- added Y1: ABM3B-32.000MHZ-8-R30-B1U-T, Personal_Project:XTAL_ABM3B-32.000MHZ-10-R30-B1U-T, F.Cu at (185.0, 85.8)
- added Z2: Diode_BZX84C6V2-7-F, Personal_Project:Diode_BZX84C6V2_SOT96P240X110-3N, F.Cu at (113.5, 99.0)
- added Z3: Diode_BZX84C6V2-7-F, Personal_Project:Diode_BZX84C6V2_SOT96P240X110-3N, F.Cu at (123.5, 85.6)
- C12: value 0p8 GRM1555C1HR80BA01D -> 2u2; footprint Capacitor_SMD:C_0402_1005Metric_Pad0.74x0.62mm_HandSolder -> Capacitor_SMD:C_0805_2012Metric
- C19: value 10n -> 0p8 GRM1555C1HR80BA01D; footprint Capacitor_SMD:C_0805_2012Metric -> Capacitor_SMD:C_0402_1005Metric_Pad0.74x0.62mm_HandSolder
- C2: value 4u7 -> 0p3 GRM1555C1HR30WA01D; footprint Capacitor_SMD:C_0805_2012Metric -> Capacitor_SMD:C_0402_1005Metric_Pad0.74x0.62mm_HandSolder
- C20: moved to F.Cu
- C21: value 100n -> 1uF
- C27: value 100n -> 4u7
- C28: value 4u7 -> 100n
- C7: value 0p3 GRM1555C1HR30WA01D -> 1u; footprint Capacitor_SMD:C_0402_1005Metric_Pad0.74x0.62mm_HandSolder -> Capacitor_SMD:C_0805_2012Metric
- C9: value 1uF -> 10n
- D1: value BZX84C4V3LT1G -> SMAJ6.0A; footprint Package_TO_SOT_SMD:SOT-23 -> Personal_Project:DO-214AC-2
- FB1: value BLM21PG601SN1D_0805 -> Part # MI0805K601R-10
- J2: value SMA PCB END LAUNCH JACK ROUND PO -> I2S_OR_LJ_OUT; footprint Personal_Project:SMA Clip Mount Adapter (top) -> Connector_PinHeader_2.54mm:PinHeader_1x03_P2.54mm_Vertical
- J3: value User Button Jumper -> SMA PCB END LAUNCH JACK ROUND PO; footprint Connector_PinHeader_2.54mm:PinHeader_1x02_P2.54mm_Vertical -> Personal_Project:SMA Clip Mount Adapter (top)
- J4: value Coin Battery Jumper -> I2C1_Headers; footprint Connector_PinHeader_2.54mm:PinHeader_1x03_P2.54mm_Vertical -> Personal_Project:PinHeader_2x03_P2.54mm_Horizontal_Court
- J5: value USB_B_Micro -> UART1_HDR; footprint Connector_USB:USB_Micro-B_XKB_U254-051T-4BH83-F1S -> Personal_Project:PinHeader_2x03_P2.54mm_Horizontal_Court
- J6: value I2C1_Headers -> I/O_HDR; footprint Connector_PinHeader_2.54mm:PinHeader_2x03_P2.54mm_Horizontal -> Connector_PinHeader_2.54mm:PinHeader_2x08_P2.54mm_Horizontal
- J7: value General_Pin_Header -> USB_C_Receptacle_USB2.0_16P; footprint Connector_PinHeader_2.54mm:PinHeader_2x07_P2.54mm_Horizontal -> Connector_USB:USB_C_Receptacle_HRO_TYPE-C-31-M-12
- LDO1: value LDO_TLV75733PDBVR -> LDO_LDLN050PU33R; footprint Personal_Project:LDO_SOT95P280X145-5N -> Package_DFN_QFN:DFN-8-1EP_3x3mm_P0.65mm_EP1.7x2.05mm
- R10: value 33R -> 10k
- R3: value 33R -> 10k; moved to F.Cu
- moved H4 174.7 mm to (196.0, 116.0)
- moved J3 166.3 mm to (197.0, 94.5), turned to 0 degrees
- moved C2 148.0 mm to (189.8, 95.2), turned to -90 degrees
- moved R3 131.1 mm to (219.5, 75.6), turned to 0 degrees
- moved J5 121.4 mm to (143.6, 77.8), turned to 90 degrees
- moved J4 114.2 mm to (154.6, 112.0), turned to -90 degrees
- moved C9 113.5 mm to (130.9, 96.5)
- moved D1 100.6 mm to (118.2, 97.5)
- moved C19 100.4 mm to (186.1, 95.2), turned to -90 degrees
- moved G*** 98.5 mm to (153.9, 88.6)
- moved Q1 97.9 mm to (123.5, 81.0), turned to 0 degrees
- moved LDO1 97.3 mm to (127.1, 96.5), turned to 180 degrees
- moved R6 93.9 mm to (119.3, 84.7)
- moved FLT1 90.7 mm to (193.0, 94.5)
- moved H1 89.9 mm to (104.0, 74.0)
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Connections:
- C12 pad 1: /RF1 -> +3.3V
- C19 pad 1: GND -> /RF, USB/RF1
- C19 pad 2: +3.3V -> GND
- C2 pad 1: /POWER_3V3 -> /RF, USB/RF_MATCH
- C20 pad 1: +3.3V -> +3.3VA
- C21 pad 1: +3.3V -> GND
- C21 pad 2: GND -> Net-(J18-Pin_1)
- C27 pad 1: +3.3V -> USB_VBUS+
- C28 pad 1: +3.3V -> /RF, USB/USB_VBUS_P+
- C7 pad 1: /RF_MATCH -> /Power_Management/VIN_LDLN050PU33R
- C9 pad 1: GND -> Net-(LDO1-FB)
- C9 pad 2: Net-(J3-Pin_1) -> GND
- D1 pad 1: GND -> /Power_Management/VIN_LDLN050PU33R
- D1 pad 2: unconnected-(D1-NC-Pad2) -> GND
- DI1 pad 1: /PB9_I2C1_SDA -> /Interfaces/I2C_SDA_HDR
- DI1 pad 2: /PB8_I2C1_SCL -> /Interfaces/I2C_SCL_HDR
- FB1 pad 1: +3.3VA -> /RF, USB/USB_VBUS_P+
- FB1 pad 2: +3.3V -> USB_VBUS+
- FLT1 pad 1: /RF_MATCH -> /RF, USB/RF_MATCH
- FLT1 pad 3: /RF_ANT -> /RF, USB/RF_ANT
- J2 pad 1: GND -> USB_VBUS+
- J2 pad 2: GND -> /Power_Management/VIN_LDLN050PU33R
- J2 pad 3: /RF_ANT -> /Power_Management/PWR+_PP
- J3 pad 1: Net-(J3-Pin_1) -> GND
- J3 pad 2: /PB5 -> GND
- J4 pad 1: +3.3V -> /Interfaces/I2C_SDA_HDR
- J4 pad 2: /VBAT -> GND
- J4 pad 3: Net-(BH1-+) -> GND
- J5 pad 1: /VBUS_5V -> GND
- J5 pad 2: /USB_D2- -> GND
- J5 pad 3: /USB_D2+ -> Net-(J5-Pin_3)
- J5 pad 4: Net-(J5-ID) -> GND
- J6 pad 1: /PB9_I2C1_SDA -> /Interfaces/I/O_HDR0
- J6 pad 3: GND -> /Interfaces/I/O_HDR1
- J6 pad 5: /PB8_I2C1_SCL -> /Interfaces/I/O_HDR2
- L1 pad 1: /RF1 -> /RF, USB/RF1
- L1 pad 2: /RF_MATCH -> /RF, USB/RF_MATCH
- LDO1 pad 1: /LDO_IN -> +3.3V
- LDO1 pad 2: GND -> unconnected-(LDO1-NC-Pad2)
- LDO1 pad 3: /LDO_IN -> Net-(LDO1-FB)
- LDO1 pad 4: unconnected-(LDO1-NC-Pad4) -> GND
- LDO1 pad 5: /LD_OUT_3V3 -> /Power_Management/VIN_LDLN050PU33R
- Q1 pad 1: /MOSFET_GATE -> /Power_Management/MOSFET_PWR
- Q1 pad 2: /EXT_POWER+_PP -> /Power_Management/PWR+_PP
- Q1 pad 3: /EXT_POWER+ -> /Power_Management/PWR+
- R10 pad 1: Net-(J15-Pin_1) -> +3.3V
- R10 pad 2: /PA2_LPUART1_TX -> /Interfaces/I2C_SCL_HDR
- R3 pad 1: /PB7_USART1_RX -> +3.3V
- R3 pad 2: Net-(J1-Pin_5) -> /Interfaces/I2C_SDA_HDR
- R6 pad 1: GND -> /Power_Management/MOSFET_PWR
- R6 pad 2: Net-(J5-ID) -> GND
- U2 pad 1: /NRST -> Net-(J18-Pin_1)
- U2 pad 2: /NRST -> Net-(J18-Pin_1)
Routing:
- net +3.3V: track 260.4 -> 2.08 mm, vias 7 -> 0
- net /NRST: track 95.1 -> 0.00 mm, vias 2 -> 0
- net /PA14_SWCLK: track 85.0 -> 0.00 mm, vias 1 -> 0
- net /PB3_SWO: track 79.4 -> 0.00 mm, vias 1 -> 0
- net /PA13_SWDIO: track 75.0 -> 0.00 mm
- net /PB5: track 67.7 -> 0.00 mm, vias 1 -> 0
- net /USB_D+: track 66.0 -> 0.00 mm
- net /USB_D-: track 66.0 -> 0.00 mm
- net /PA1: track 53.2 -> 0.00 mm, vias 1 -> 0
- net /VBAT: track 51.4 -> 0.00 mm
- net /PA4_SPI1_NSS: track 51.2 -> 0.00 mm, vias 1 -> 0
- net /PA0: track 48.8 -> 0.00 mm, vias 1 -> 0
- net /PB7_USART1_RX: track 48.3 -> 0.00 mm, vias 1 -> 0
- net /PB4: track 46.5 -> 0.00 mm, vias 1 -> 0
- net /PB6_USART1_TX: track 46.1 -> 0.00 mm, vias 1 -> 0
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- added copper zone on F.Cu, net +3.3V
- added copper zone on F.Cu, net +3.3VA
- added copper zone on F.Cu, net /Power_Management/MOSFET_PWR
- added copper zone on F.Cu, net /Power_Management/PWR+
- added copper zone on F.Cu, net /Power_Management/PWR+_PP
- added copper zone on F.Cu, net /Power_Management/VIN_LDLN050PU33R
- added copper zone on F.Cu, net /RF, USB/USB_VBUS_P+
- added copper zone on F.Cu, net USB_VBUS+
- removed copper zone on F.Cu, net /EXT_POWER+
- removed copper zone on F.Cu, net /EXT_POWER+_PP
- removed copper zone on F.Cu, net /LDO_IN
- removed copper zone on F.Cu, net /MOSFET_GATE
- removed copper zone on F.Cu, net /POWER_3V3
- removed copper zone on B.Cu, net GND
- removed copper zone on In1.Cu, net GND
- removed copper zone on In2.Cu, net GND
Other:
- board text added: "VBUS/PWR"
- board text removed: "3V3"
- board text removed: "A0"
- board text removed: "A1"
- board text removed: "A10"
- board text removed: "A15"
- board text removed: "A5CK"
- board text removed: "A6MI"
- board text removed: "A7MO"
- board text removed: "A8M"
- board text removed: "A9"
- board text removed: "B0"
- board text removed: "B1"
- board text removed: "B2"
- board text removed: "B4"
- board text removed: "B5"
- board text removed: "BTN ACT"
- board text removed: "E4"
- board text removed: "EXTNOLDO"
- board text removed: "EXTWLDO"
- board text removed: "GN"
- board text removed: "GND/BOOT/3V3"
- board text removed: "I2C1"
- board text removed: "INT/EXT"
- board text removed: "LDO/NOLDO"
- board text removed: "LPUART1"
- board text removed: "NRST"
- board text removed: "ON/OFF"
- board text removed: "PA2TX"
- board text removed: "PA3RX"
- board text removed: "PB6TX"
- board text removed: "PB7RX"
- board text removed: "PB8CL"
- board text removed: "PB9SDA"
- board text removed: "POWER"
- board text removed: "SIO/NR/SO/CL"
- board text removed: "SPI1"
- board text removed: "SPI1NSS"
- board text removed: "USART1"
- board text removed: "USR BTN"
- board text removed: "V+"
- board text removed: "V-"
- board text removed: "VBAT"
- board text removed: "VBUS5V"

Commit message: Update
Parts:
- DI1, R5: moved to B.Cu
- moved J5 34.9 mm to (137.6, 112.3), turned to -90 degrees
- moved R5 28.7 mm to (135.1, 108.5)
- moved J6 12.5 mm to (145.3, 77.9)
- moved G*** 9.06 mm to (145.0, 86.9)
- moved C3 5.18 mm to (175.1, 86.6)
- moved C16 5.00 mm to (169.8, 106.5), turned to 90 degrees
- moved C5 1.75 mm to (175.1, 88.9)
- moved DI1 1.55 mm to (152.0, 108.1), turned to 90 degrees
- moved C11 0.51 mm to (171.0, 95.0)
- moved C4 0.46 mm to (175.1, 84.3)
- moved C14 0.45 mm to (173.9, 101.6)
- moved C13 0.35 mm to (170.8, 100.9)
- moved J4 0.31 mm to (154.6, 112.3)
- moved C8 0.15 mm to (187.0, 90.0)
- moved C6 0.10 mm to (189.5, 90.0)
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Connections:
- IC2 pad 37: /RF, USB/USB_D2-_DI -> /RF, USB/USB_DI_D2-
- IC2 pad 38: /RF, USB/USB_D2+_DI -> /RF, USB/USB_DI_D2+
- U5 pad 1: /RF, USB/USB_D2-_DI -> /RF, USB/USB_DI_D2+
- U5 pad 3: /RF, USB/USB_D2+_DI -> /RF, USB/USB_DI_D2-
- U5 pad 4: /RF, USB/USB_D2+ -> /RF, USB/USB_D2-
- U5 pad 6: /RF, USB/USB_D2- -> /RF, USB/USB_D2+
Routing:
- net /RF, USB/USB_DI_D2-: track 0.00 -> 66.3 mm
- net /RF, USB/USB_DI_D2+: track 0.00 -> 66.3 mm
- net +3.3V: track 2.08 -> 18.0 mm
- net /STM32WB55CGU6/OSC_OUT: track 0.00 -> 11.2 mm
- net /STM32WB55CGU6/SMPS_FB: track 0.00 -> 10.2 mm
- net GND: track 0.00 -> 9.50 mm, vias 0 -> 4
- net /RF, USB/USB_D2+: track 0.00 -> 9.11 mm
- net /RF, USB/USB_D2-: track 0.00 -> 7.37 mm
- net /STM32WB55CGU6/OSC_IN: track 0.00 -> 5.70 mm
- net /Interfaces/I/O_HDR6: track 0.00 -> 5.18 mm, vias 0 -> 1
- net /RF, USB/RF1: track 0.00 -> 4.73 mm
- net Net-(IC2-PC14-OSC32_IN): track 0.00 -> 4.41 mm
- net /Interfaces/I/O_HDR3: track 0.00 -> 4.30 mm, vias 0 -> 1
- net /RF, USB/RF_MATCH: track 0.00 -> 3.84 mm
- net /Interfaces/USR_BTN: track 0.00 -> 3.80 mm, vias 0 -> 1
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
Commit message: Update
Parts:
- removed BH2: Battery_Holder_1060TR, Personal_Project:Battery_Holder_1060TR
- removed FPC2: FPC_0545482072, Personal_Project:FPC_0545482072
- removed J18: User Button Jumper, Connector_PinHeader_2.54mm:PinHeader_1x02_P2.54mm_Vertical
- removed J6: I/O_HDR, Connector_PinHeader_2.54mm:PinHeader_2x08_P2.54mm_Horizontal
- removed J9: Coin Battery Jumper, Connector_PinHeader_2.54mm:PinHeader_1x03_P2.54mm_Vertical
- added C17: 100n, Capacitor_SMD:C_0805_2012Metric, F.Cu at (162.7, 78.3)
- added G***: LOGO, Personal_Project:PCB_Logo, B.Cu at (183.0, 77.8)
- added J1: I/O_HDR, Connector_PinHeader_2.54mm:PinHeader_2x05_P2.54mm_Horizontal, F.Cu at (130.4, 112.4)
- added MEM1: MX35LF2G24AD-Z4I, Package_DFN_QFN:WDFN-8-1EP_8x6mm_P1.27mm_EP6x4.8mm, F.Cu at (155.3, 80.4)
- added R1: 33R, Resistor_SMD:R_0805_2012Metric, F.Cu at (148.3, 79.7)
- added R11: 33R, Resistor_SMD:R_0805_2012Metric, F.Cu at (159.0, 85.7)
- added R12: 33R, Resistor_SMD:R_0805_2012Metric, F.Cu at (148.3, 82.0)
- added R2: 33R, Resistor_SMD:R_0805_2012Metric, F.Cu at (162.1, 81.2)
- added R9: 33R, Resistor_SMD:R_0805_2012Metric, F.Cu at (162.1, 83.4)
- DI1, R5: moved to F.Cu
- moved R10 75.4 mm to (149.3, 109.0)
- moved R3 71.2 mm to (156.7, 109.0), turned to 180 degrees
- moved C15 51.6 mm to (184.2, 110.4), turned to 0 degrees
- moved FB2 45.6 mm to (181.2, 109.7), turned to -90 degrees
- moved C18 42.6 mm to (182.1, 106.7), turned to 0 degrees
- moved C20 40.0 mm to (182.1, 104.4), turned to 0 degrees
- moved R5 30.9 mm to (165.0, 100.9), turned to -90 degrees
- moved J11 22.7 mm to (145.2, 102.7), turned to 90 degrees
- moved G*** 13.5 mm to (134.8, 78.0)
- moved C21 4.36 mm to (113.6, 113.8), turned to 0 degrees
- moved J5 4.26 mm to (141.9, 112.4)
- moved C3 2.05 mm to (173.1, 86.6)
- moved C4 2.05 mm to (173.1, 84.3)
- moved C5 2.05 mm to (173.1, 88.9)
- moved C1 1.90 mm to (178.0, 81.7)
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Connections:
- net /RF, USB/USB_VBUS_P+ renamed /RF, USB/VBUS_P+
- net USB_VBUS+ renamed VBUS+
- C14 pad 1: /STM32WB55CGU6/VBAT -> +3.3V
- C21 pad 2: Net-(J18-Pin_1) -> /Interfaces/USR_BTN
- IC2 pad 1: /STM32WB55CGU6/VBAT -> +3.3V
- IC2 pad 10: /Interfaces/I/O_HDR1 -> /STM32WB55CGU6/PA1
- IC2 pad 11: /Interfaces/QSPI_CS0 -> /STM32WB55CGU6/PA2_QUADSPI_BK1_NCS
- IC2 pad 12: /Interfaces/QSPI_CLK -> /STM32WB55CGU6/PA3_QUADSPI_CLK
- IC2 pad 15: /Interfaces/QSPI_IO3 -> /STM32WB55CGU6/PA6_QUADSPI_BK1_IO3
- IC2 pad 16: /Interfaces/QSPI_IO2 -> /STM32WB55CGU6/PA7_QUADSPI_BK1_IO2
- IC2 pad 17: /Interfaces/I/O_HDR7 -> /Interfaces/I/O_HDR1
- IC2 pad 19: /Interfaces/I/O_HDR4 -> /STM32WB55CGU6/PB2
- IC2 pad 28: /Interfaces/USR_BTN -> /Interfaces/I/O_HDR4
- IC2 pad 30: /Interfaces/I/O_HDR6 -> /Interfaces/I/O_HDR2
- IC2 pad 42: /Interfaces/I/O_HDR2 -> /Interfaces/USR_BTN
- IC2 pad 47: /Interfaces/I/O_HDR5 -> /Interfaces/I/O_HDR0
- IC2 pad 5: /Interfaces/QSPI_IO1 -> /STM32WB55CGU6/PB8_QUADSPI_BK1_IO1
- IC2 pad 6: /Interfaces/QSPI_IO0 -> /STM32WB55CGU6/PB9_QUADSPI_BK1_IO0
- IC2 pad 9: /Interfaces/I/O_HDR0 -> /STM32WB55CGU6/PA0
- R4 pad 1: Net-(OS1-OUTPUT) -> Net-(IC2-PC14-OSC32_IN)
- R4 pad 2: Net-(IC2-PC14-OSC32_IN) -> Net-(OS1-OUTPUT)
- U2 pad 1: Net-(J18-Pin_1) -> /Interfaces/USR_BTN
- U2 pad 2: Net-(J18-Pin_1) -> /Interfaces/USR_BTN
Routing:
- net +3.3V: track 18.0 -> 261.6 mm, vias 0 -> 14
- net /Interfaces/NRST: track 5.98 -> 129.3 mm, vias 0 -> 5
- net /Interfaces/I/O_HDR4: track 0.00 -> 114.7 mm, vias 0 -> 2
- net /Interfaces/I/O_HDR2: track 0.00 -> 107.6 mm, vias 0 -> 2
- net /Interfaces/I/O_HDR3: track 4.30 -> 110.7 mm, vias 1 -> 2
- net /Interfaces/I2C_SCL_HDR: track 0.00 -> 93.5 mm, vias 0 -> 2
- net /Interfaces/SWO: track 0.00 -> 93.3 mm, vias 0 -> 1
- net /Interfaces/I/O_HDR1: track 0.00 -> 92.1 mm, vias 0 -> 1
- net /Interfaces/SWDIO: track 0.00 -> 83.6 mm, vias 0 -> 1
- net /Interfaces/SWCLK: track 0.00 -> 80.4 mm, vias 0 -> 1
- net /Interfaces/USR_BTN: track 3.80 -> 82.7 mm, vias 1 -> 2
- net /STM32WB55CGU6/PB8_QUADSPI_BK1_IO1: track 0.00 -> 71.8 mm, vias 0 -> 2
- net /STM32WB55CGU6/PA7_QUADSPI_BK1_IO2: track 0.00 -> 71.8 mm, vias 0 -> 2
- net /STM32WB55CGU6/PA2_QUADSPI_BK1_NCS: track 0.00 -> 71.4 mm, vias 0 -> 2
- net /Interfaces/I/O_HDR0: track 0.00 -> 59.8 mm, vias 0 -> 1
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- added copper zone on In2.Cu, net +3.3V
- added copper zone on B.Cu, net GND
- added copper zone on In1.Cu, net GND
- added copper zone on In2.Cu, net GND
Other:
- board text added: "3V3"
- board text added: "Bluetooth Board Revision: REV B Designer: Peter Hancak MCU: STM32WB55CGU6 LDO: LDLN050PU33R VIN: 2.7 to 6.5V"
- board text added: "I2C"
- board text added: "PA8-MCO"
- board text added: "PB0"
- board text added: "PB1"
- board text added: "PB7"
- board text added: "PE4"
- board text added: "PH3-BOOT0"
- board text added: "ROM FLS"
- board text added: "SCL"
- board text added: "SD NR SO SC"
- board text added: "SDA"
- board text added: "SPI"
- board text added: "TX/RX"
- board text added: "UART"
- board text added: "USB JST1"
- board text added: "USR BTN"
- board text added: "VIN:2.7 to 6.5V"
- board text removed: "VBUS/PWR"

Commit message: Update
Parts:
- removed C26, C28: 100n, Capacitor_SMD:C_0805_2012Metric
- removed FB1: Part # MI0805K601R-10, Capacitor_SMD:C_0805_2012Metric
- moved G*** 5.40 mm to (183.2, 83.2)
- moved C27 0.58 mm to (106.9, 92.6)
Connections:
- J7 pad A4: /RF, USB/VBUS_P+ -> VBUS+
- J7 pad A9: /RF, USB/VBUS_P+ -> VBUS+
- J7 pad B4: /RF, USB/VBUS_P+ -> VBUS+
- J7 pad B9: /RF, USB/VBUS_P+ -> VBUS+
- U5 pad 5: /RF, USB/VBUS_P+ -> VBUS+
- Z2 pad 3: /RF, USB/VBUS_P+ -> VBUS+
Routing:
- net VBUS+: track 0.00 -> 19.2 mm, vias 0 -> 3
- net /RF, USB/VBUS_P+: track 19.2 -> 0.00 mm, vias 3 -> 0
- removed copper zone on F.Cu, net /RF, USB/VBUS_P+
Other:
- rule pad_to_mask_clearance: 0.038 -> 0

Commit message: Update
Parts:
- removed Y1: ABM3B-32.000MHZ-8-R30-B1U-T, Personal_Project:XTAL_ABM3B-32.000MHZ-10-R30-B1U-T
- added C23: 1n, Capacitor_SMD:C_0805_2012Metric, F.Cu at (193.1, 99.0)
- added C28: 100n, Capacitor_SMD:C_0805_2012Metric, F.Cu at (197.8, 95.1)
- added OS2: Oscillator_ATX-11-F-32.000MHZ-F05-T, Personal_Project:Oscillator_ECSTXO32CSMV320ANTR, F.Cu at (194.2, 95.1)
- FPC1: value FPC_0545481072 -> FPC_10051922-1010ELF; footprint Personal_Project:FPC_0545481072 -> Personal_Project:FPC_10051922_1010
- moved FPC1 14.4 mm to (177.3, 126.6), turned to 180 degrees
- moved G*** 14.2 mm to (143.3, 89.4)
- moved C12 14.1 mm to (137.6, 109.7)
- moved R6 14.1 mm to (129.3, 94.7)
- moved C1 14.1 mm to (188.0, 91.7)
- moved C10 14.1 mm to (197.8, 108.8)
- moved C11 14.1 mm to (179.5, 104.5)
- moved C13 14.1 mm to (180.8, 111.5)
- moved C14 14.1 mm to (183.9, 112.2)
- moved C15 14.1 mm to (194.2, 120.4)
- moved C16 14.1 mm to (179.2, 117.0)
- moved C17 14.1 mm to (172.7, 88.3)
- moved C18 14.1 mm to (192.1, 116.7)
- moved C19 14.1 mm to (196.1, 105.2)
- moved C2 14.1 mm to (199.8, 105.2)
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Connections:
- IC2 pad 24: /STM32WB55CGU6/OSC_OUT -> unconnected-(IC2-OSC_OUT-Pad24)
Routing:
- net /STM32WB55CGU6/OSC_OUT: track 11.2 -> 0.00 mm
- net +3.3V: track 261.6 -> 267.9 mm, vias 14 -> 15
- net /STM32WB55CGU6/OSC_IN: track 5.70 -> 2.81 mm
- net /STM32WB55CGU6/OSC_OUTPUT: track 0.00 -> 2.15 mm
- net /Interfaces/SPI_MISO: track 37.7 -> 39.1 mm
- net GND: track 41.1 -> 41.6 mm, vias 244 -> 248
Other:
- board text added: "BOOT0"
- board text added: "GND"
- board text added: "HIGH LOW"
- board text added: "NRST"
- board text added: "PWR SRC"
- board text added: "PWR+"
- board text added: "RST"
- board text added: "SWCLK"
- board text added: "SWDIO"
- board text added: "SWO"
- board text added: "USB-C"
- board text added: "VIN:4.0 to 6.5V"
- board text removed: "VIN:2.7 to 6.5V"

Commit message: Update
Parts:
- moved C12 14.1 mm to (127.5, 99.7)
- moved R6 14.1 mm to (119.3, 84.7)
- moved C1 14.1 mm to (178.0, 81.7)
- moved C10 14.1 mm to (187.8, 98.8)
- moved C11 14.1 mm to (169.5, 94.5)
- moved C13 14.1 mm to (170.8, 101.5)
- moved C14 14.1 mm to (173.9, 102.2)
- moved C15 14.1 mm to (184.2, 110.4)
- moved C16 14.1 mm to (169.2, 107.0)
- moved C17 14.1 mm to (162.7, 78.3)
- moved C18 14.1 mm to (182.1, 106.7)
- moved C19 14.1 mm to (186.1, 95.2)
- moved C2 14.1 mm to (189.8, 95.2)
- moved C20 14.1 mm to (182.1, 104.4)
- moved C21 14.1 mm to (113.6, 113.8)
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Routing:
- net GND: track 41.6 -> 215.1 mm
- net +3.3V: track 267.9 -> 128.9 mm
- net /STM32WB55CGU6/BOOT0: track 50.3 -> 157.7 mm
- net /STM32WB55CGU6/PA7_QUADSPI_BK1_IO2: track 71.8 -> 12.5 mm
- net /STM32WB55CGU6/PA6_QUADSPI_BK1_IO3: track 50.3 -> 12.8 mm
- net /Interfaces/I/O_HDR3: track 110.7 -> 97.9 mm
- net /Interfaces/I/O_HDR2: track 107.6 -> 94.8 mm
- net /Interfaces/I/O_HDR4: track 114.7 -> 101.9 mm
- net /Interfaces/NRST: track 129.3 -> 122.5 mm

Commit message: Update
Routing:
- net GND: track 215.1 -> 41.6 mm
- net +3.3V: track 128.9 -> 267.9 mm
- net /STM32WB55CGU6/BOOT0: track 157.7 -> 50.3 mm
- net /STM32WB55CGU6/PA7_QUADSPI_BK1_IO2: track 12.5 -> 71.8 mm
- net /STM32WB55CGU6/PA6_QUADSPI_BK1_IO3: track 12.8 -> 50.3 mm
- net /Interfaces/I/O_HDR3: track 97.9 -> 110.7 mm
- net /Interfaces/I/O_HDR2: track 94.8 -> 107.6 mm
- net /Interfaces/I/O_HDR4: track 101.9 -> 114.7 mm
- net /Interfaces/NRST: track 122.5 -> 129.3 mm
