File: Bluetooth_Board.kicad_sch (KiCad schematic)
At the start: 57 parts, among them J1 5V Power Pins, J11 3V3 Power Pins, J12 GPIO_Connector, J13 3V3 Power Source Jumpers, J14 Debug_Pins, J16 61302021821, J18 GPIO_Connector, J19 Power Select Jumpers, J2 SMA PCB END LAUNCH JACK ROUND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, J3 User Button Jumper, J5 Power Pins, J6 USB_B_Micro, J7 BOOT0_Jumper, J9 LCD_I2C3_Connector, U1 STM32WB55RGVx, U3 USBLC6-2SC6, Y1 ABM3B-32.000MHZ-10-R30-B1U-T, Y2 Clock_ECS-327MVATX-7-CN-TR

Commit message: Update
Parts:
- added IC1: STM32WB55CGU6, Personal_Project:STM32WB55CGU6_QFN50P700X700X60-49N-D, symbol Personal_Projects:STM32WB55CGU6
Other:
- note added: "STM32MP157FAD1 2x STM32WB55CGU6 2x STM32WB5MMGH6TR STM32MP135DAF7 STM32H7S7L8H6H STSPIN958TR STM32H7S3I8T6 LSM6DSV16XTR ISM330BXTR STM32WL55CCU6 STM32WL55JCI6 2x"
Changed lines of the file:
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@@
 		)
 	)
+	(text "STM32MP157FAD1 2x\nSTM32WB55CGU6 2x\nSTM32WB5MMGH6TR\nSTM32MP135DAF7\nSTM32H7S7L8H6H\n\nSTSPIN958TR\nSTM32H7S3I8T6\nLSM6DSV16XTR\nISM330BXTR\nSTM32WL55CCU6\nSTM32WL55JCI6 2x"
+		(exclude_from_sim no)
+		(at -16.51 29.21 0)
+		(effects
+			(font
+				(size 1 1)
+			)
+		)
+	)
 	(text "The load capacitances are integrated on chip and \ncan be tuned according to the selected crystal via \nan internal register. By default, the load capacitances \nare 8 pF for the NX2016 from NDK used on the boards.\n\nRCC clock HSE register (RCC_HSECR)\nBits 13:8 HSETUNE[5:0]: HSE capacitor tuning\nCan be changed by software. Do not change when HSE is on.\n0x00: minimum load capacitance\n0x3F maximum load capacitance"
 		(exclude_from_sim no)
@@
 					(unit 1)
 				)
+			)
+		)
+	)
+	(symbol
+		(lib_id "Personal_Projects:STM32WB55CGU6")
+		(at 226.06 207.01 0)
+		(unit 1)
+		(exclude_from_sim no)
+		(in_bom yes)
+		(on_board yes)
+		(dnp no)
+		(fields_autoplaced yes)
+		(property "Reference" "IC1"
+			(at 274.32 200.6914 0)
+			(effects
+				(font
+					(size 1.27 1.27)
+				)
+			)
+		)
+		(property "Value" "STM32WB55CGU6"
+			(at 274.32 203.2314 0)
+			(effects
+				(font
+					(size 1.27 1.27)
+				)
+			)
+		)
+		(property "Footprint" "Personal_Project:STM32WB55CGU6_QFN50P700X700X60-49N-D"
+			(at 267.97 291.77 0)
+			(effects
+				(font
+					(size 1.27 1.27)
+				)
+				(justify left top)
+				(hide yes)
+			)
+		)
+		(property "Datasheet" "https://www.st.com/en/microcontrollers/stm32wb55cg.html"
+			(at 267.97 391.77 0)
+			(effects
+				(font
+					(size 1.27 1.27)
+				)
+				(justify left top)
+				(hide yes)
+			)
+		)
+		(property "Description" "ARM Microcontrollers - MCU Ultra-low-power dual core Arm Cortex-M4 MCU 64 MHz, Cortex-M0 32MHz with 1 Mbyte Flash, BLE, 802.15.4, USB, LCD, AES-256"
+			(at 241.046 283.464 0)
+			(effects
+				(font
+					(size 1.27 1.27)
+				)
+				(hide yes)
+			)
+		)
+		(property "Height" "0.6"
+			(at 267.97 591.77 0)
+			(effects
+				(font
+					(size 1.27 1.27)
+				)
+				(justify left top)
+				(hide yes)
+			)
+		)
+		(property "Mouser Part Number" "511-STM32WB55CGU6"
+			(at 267.97 691.77 0)
+			(effects
+				(font
+					(size 1.27 1.27)
+				)
+				(justify left top)
+				(hide yes)
+			)
+		)
+		(property "Mouser Price/Stock" "https://www.mouser.co.uk/ProductDetail/STMicroelectronics/STM32WB55CGU6?qs=lYGu3FyN48eI3bRY%252B36gew%3D%3D"
+			(at 267.97 791.77 0)
+			(effects
+				(font
+					(size 1.27 1.27)
+				)
+				(justify left top)
+				(hide yes)
+			)
+		)
+		(property "Manufacturer_Name" "STMicroelectronics"
+			(at 267.97 891.77 0)
+			(effects
+				(font
+					(size 1.27 1.27)
+				)
+				(justify left top)
+				(hide yes)
+			)
+		)
+		(property "Manufacturer_Part_Number" "STM32WB55CGU6"
+			(at 267.97 991.77 0)
+			(effects
+				(font
+					(size 1.27 1.27)
+				)
+				(justify left top)
+				(hide yes)
+			)
+		)
+		(pin "19"
+		)
+		(pin "2"
+		)
+		(pin "35"
+		)
+		(pin "36"
+		)
+		(pin "37"
+		)
+		(pin "33"
+		)
+		(pin "34"
+		)
+		(pin "22"
+		)
+		(pin "23"
+		)
+		(pin "20"
+		)
+		(pin "21"
+		)
+		(pin "1"
+		)
+		(pin "17"
+		)
+		(pin "18"
+		)
+		(pin "3"
+		)
+		(pin "30"
+		)
+		(pin "31"
+		)
+		(pin "32"
+		)
+		(pin "15"
+		)
+		(pin "16"
+		)
+		(pin "14"
+		)
+		(pin "11"
+		)
+		(pin "13"
+		)
+		(pin "28"
+		)
+		(pin "29"
+		)
+		(pin "12"
+		)
+		(pin "10"
+		)
+		(pin "26"
+		)
+		(pin "27"
+		)
+		(pin "24"
+		)
+		(pin "25"
+		)
+		(pin "38"
+		)
+		(pin "39"
+		)
+		(pin "4"
+		)
+		(pin "40"
+		)
+		(pin "41"
+		)
+		(pin "42"
+		)
+		(pin "43"
+		)
+		(pin "44"
+		)
+		(pin "45"
+		)
+		(pin "46"
+		)
+		(pin "47"
+		)
+		(pin "48"
+		)
+		(pin "49"
+		)
+		(pin "5"
+		)
+		(pin "6"
+		)
+		(pin "7"
+		)
+		(pin "8"
+		)
+		(pin "9"
+		)
+		(instances
+			(project ""
+				(path "/05989bb3-969e-4aaa-b344-5f0e2d5af968"
+					(reference "IC1")
+					(unit 1)
+				)

Commit message: Update
Parts:
- removed C1, C17, C18, C6: 4u7, Capacitor_SMD:C_0805_2012Metric_Pad1.18x1.45mm_HandSolder, symbol Device:C
- removed C10, C11, C14, C15, C16, C3, C5, C8: 100n, Capacitor_SMD:C_0805_2012Metric_Pad1.18x1.45mm_HandSolder, symbol Device:C
- removed C13: 1u, Capacitor_SMD:C_0805_2012Metric_Pad1.18x1.45mm_HandSolder, symbol Device:C
- removed C2: 10n, Capacitor_SMD:C_0805_2012Metric_Pad1.18x1.45mm_HandSolder, symbol Device:C
- removed C4: 1uF, Capacitor_SMD:C_0805_2012Metric_Pad1.18x1.45mm_HandSolder, symbol Device:C
- removed FB1: FCM1608KF-601T03, Inductor_SMD:L_0603_1608Metric_Pad1.05x0.95mm_HandSolder, symbol Device:FerriteBead
- removed J12: GPIO_Connector, Connector_PinHeader_2.54mm:PinHeader_2x11_P2.54mm_Vertical, symbol Connector_Generic:Conn_02x11_Odd_Even
- removed J16: 61302021821, Personal_Project:WR-PHD 2.54 MM DUAL SOCKET HEADE, symbol Personal_Projects:WR-PHD 2.54 MM DUAL SOCKET HEADE
- removed J18: GPIO_Connector, Connector_PinHeader_2.54mm:PinHeader_2x10_P2.54mm_Vertical, symbol Connector_Generic:Conn_02x11_Odd_Even
- removed J7: BOOT0_Jumper, Connector_PinHeader_2.54mm:PinHeader_1x03_P2.54mm_Vertical, symbol Connector:Conn_01x03_Pin
- removed J9: LCD_I2C3_Connector, Connector_PinHeader_2.54mm:PinHeader_1x04_P2.54mm_Vertical, symbol Connector:Conn_01x04_Pin
- removed L2: 10u Murata LQM21FN100M70L, Inductor_SMD:L_0805_2012Metric_Pad1.15x1.40mm_HandSolder, symbol Device:L
- removed L3: 10n Murata LQG15WZ10NJ02D, Inductor_SMD:L_0402_1005Metric_Pad0.77x0.64mm_HandSolder, symbol Device:L
- removed R1: 10R, Resistor_SMD:R_0805_2012Metric_Pad1.20x1.40mm_HandSolder, symbol Device:R
- removed U1: STM32WB55RGVx, Package_DFN_QFN:QFN-68-1EP_8x8mm_P0.4mm_EP6.4x6.4mm, symbol MCU_ST_STM32WB:STM32WB55RGVx
- removed U5: ~, Personal_Project:Button_KMR231GLFS, symbol Personal_Projects:Button_KMR231GLFS
- removed Y1: ABM3B-32.000MHZ-10-R30-B1U-T, Personal_Project:XTAL_ABM3B-32.000MHZ-10-R30-B1U-T, symbol Personal_Projects:ABM3B-32.000MHZ-10-R30-B1U-T
- removed Y2: Clock_ECS-327MVATX-7-CN-TR, Personal_Project:Clock_ECS327MVATX7CNTR, symbol Personal_Projects:Clock_ECS-327MVATX-7-CN-TR
- added BH1: Battery_Holder_1060TR, Personal_Project:Battery_Holder_1060TR, symbol Personal_Projects:Battery_Holder_1060TR
- added C19: 10n, Capacitor_SMD:C_0805_2012Metric_Pad1.18x1.45mm_HandSolder, symbol Device:C
- added C20, C21, C22, C27, C29, C30, C33, C34: 100n, Capacitor_SMD:C_0805_2012Metric_Pad1.18x1.45mm_HandSolder, symbol Device:C
- added C23, C26, C28, C31, C32: 4u7, Capacitor_SMD:C_0805_2012Metric_Pad1.18x1.45mm_HandSolder, symbol Device:C
- added C35: 1u, Capacitor_SMD:C_0805_2012Metric_Pad1.18x1.45mm_HandSolder, symbol Device:C
- added C36: 1uF, Capacitor_SMD:C_0805_2012Metric_Pad1.18x1.45mm_HandSolder, symbol Device:C
- added FB2: FCM1608KF-601T03, Inductor_SMD:L_0603_1608Metric_Pad1.05x0.95mm_HandSolder, symbol Device:FerriteBead
- added J10: LPUART1_Header, Connector_PinHeader_2.54mm:PinHeader_1x04_P2.54mm_Vertical, symbol Connector_Generic:Conn_01x04
- added J15: USART1_Header, Connector_PinHeader_2.54mm:PinHeader_1x04_P2.54mm_Vertical, symbol Connector_Generic:Conn_01x04
- added J16: Pin_Header, Connector_PinHeader_2.54mm:PinHeader_2x07_P2.54mm_Vertical, symbol Connector_Generic:Conn_02x07_Odd_Even
- added J20: SPI1_Header, Connector_PinHeader_2.54mm:PinHeader_1x06_P2.54mm_Vertical, symbol Connector_Generic:Conn_01x06
- added J4: Coin Battery Jumper, Connector_PinHeader_2.54mm:PinHeader_1x03_P2.54mm_Vertical, symbol Connector_Generic:Conn_01x03
- added J7: I2C3_Header, Connector_PinHeader_2.54mm:PinHeader_1x04_P2.54mm_Vertical, symbol Connector_Generic:Conn_01x04
- added J8: BOOT0_Jumper, Connector_PinHeader_2.54mm:PinHeader_1x03_P2.54mm_Vertical, symbol Connector:Conn_01x03_Pin
- added J9: I2C1_Header, Connector_PinHeader_2.54mm:PinHeader_1x04_P2.54mm_Vertical, symbol Connector_Generic:Conn_01x04
- added L4: 10u Murata LQM21FN100M70L, Inductor_SMD:L_0805_2012Metric_Pad1.15x1.40mm_HandSolder, symbol Device:L
- added L5: 10n Murata LQG15WZ10NJ02D, Inductor_SMD:L_0402_1005Metric_Pad0.77x0.64mm_HandSolder, symbol Device:L
- added R2: 10R, Resistor_SMD:R_0805_2012Metric_Pad1.20x1.40mm_HandSolder, symbol Device:R
- added U2: ~, Personal_Project:Button_KMR231GLFS, symbol Personal_Projects:Button_KMR231GLFS
- added Y3: Clock_ECS-327MVATX-7-CN-TR, Personal_Project:Clock_ECS327MVATX7CNTR, symbol Personal_Projects:Clock_ECS-327MVATX-7-CN-TR
- added Y4: ABM3B-32.000MHZ-8-R30-B1U-T, Personal_Project:XTAL_ABM3B-32.000MHZ-10-R30-B1U-T, symbol Personal_Projects:ABM3B-32.000MHZ-10-R30-B1U-T
Connections:
- net SWCLK is gone; now on net PA14_SWCLK: J14.4 (Pin_4)
- net SWDIO is gone; now on net PA13_SWDIO: J14.2 (Pin_2)
- net SWO is gone; now on net PB3_SWO: J14.6 (Pin_6)
- net USB_D+ is gone; now on net PA12_USB_D+: U3.4 (I/O2)
- net USB_D- is gone; now on net PA11_USB_D-: U3.6 (I/O1)
- net +3.3V: now also IC1.20 (VDD_1), IC1.23 (VDDRF), IC1.34 (VDDSMPS), IC1.35 (VDD_2), IC1.40 (VDDUSB), IC1.48 (VDD_3), C19.2, C20.1, C21.1, C22.1, C26.1, C27.1, C28.1, C29.1, C32.1, C33.1, FB2.1, J10.1 (Pin_1), J15.1 (Pin_1), J20.1 (Pin_1), J4.1 (Pin_1), J7.1 (Pin_1), J8.1 (Pin_1), J9.1 (Pin_1), Y3.4 (VDD)
- net +3.3VA: now also IC1.8 (VDDA), C34.1, C35.1, FB2.2
- net +5V: now also C23.1
- net BOOT0: now also IC1.4 (PH3-BOOT0), J8.2 (Pin_2)
- net GND: now also IC1.22 (VSSRF), IC1.32 (VSSSMPS), IC1.49 (GND), BH1.2 (-), C19.1, C20.2, C21.2, C22.2, C23.2, C26.2, C27.2, C28.2, C29.2, C30.2, C31.2, C32.2, C33.2, C34.2, C35.2, C36.1, J10.2 (Pin_2), J15.2 (Pin_2), J16.1 (Pin_1), J20.2 (Pin_2), J7.2 (Pin_2), J8.3 (Pin_3), J9.2 (Pin_2), U2.3, U2.4, U2.5 (GND), Y3.2 (GND), Y4.2, Y4.4
- net NRST: now also IC1.7 (NRST), C36.2, U2.1, U2.2
- net PA0: now also IC1.9 (PA0), J3.2 (Pin_2), J16.5 (Pin_5)
- net PA15: now also IC1.42 (PA15), J16.9 (Pin_9)
- net PA2_LPUART1_TX: now also IC1.11 (PA2), J10.3 (Pin_3)
- net PA3_LPUART1_RX: now also IC1.12 (PA3), J10.4 (Pin_4)
- net PA5: now also IC1.14 (PA5), J16.4 (Pin_4)
- net PA8_MCO: now also IC1.17 (PA8), J16.3 (Pin_3)
- net PB0: now also IC1.28 (PB0), J16.12 (Pin_12)
- net PB1: now also IC1.29 (PB1), J16.11 (Pin_11)
- net PB2: now also IC1.19 (PB2), J16.2 (Pin_2)
- net PB8_I2C1_SCL: now also IC1.5 (PB8), J9.3 (Pin_3); no longer J3.2 (Pin_2)
- net PB9_I2C1_SDA: now also IC1.6 (PB9), J9.4 (Pin_4)
- net PC15-OSC32_OUT: now also IC1.3 (PC15-OSC32_OUT), J16.6 (Pin_6)
- net PE4: now also IC1.30 (PE4), J16.10 (Pin_10)
- net RF1: now also IC1.21 (RF1)
- net SMPS_FB: now also IC1.31 (VFBSMPS), C31.1, L4.1
- net SMPS_LX: now also IC1.33 (VLXSMPS), L5.2
- net SMPS_LXL: now also L4.2, L5.1
- net VBAT: now reaches IC1.1 (VBAT)
- net VBAT: now also C30.1, J4.2 (Pin_2)
- net PA1_SPI1_SCK: now reaches IC1.10 (PA1)
- net PA1_SPI1_SCK: now also J20.3 (Pin_3)
- net PA4_SPI1_NSS: now reaches IC1.13 (PA4)
- net PA4_SPI1_NSS: now also J20.6 (Pin_6)
- net PA6_SPI1_MISO: now reaches IC1.15 (PA6)
- net PA6_SPI1_MISO: now also J20.4 (Pin_4)
- net PA7_I2C3_SCL: now reaches IC1.16 (PA7)
- net PA7_I2C3_SCL: now also J7.3 (Pin_3)
- net PA9_USART1_TX: now reaches IC1.18 (PA9)
- net PA9_USART1_TX: now also J15.3 (Pin_3)
- net at IC1.2 (PC14-OSC32_IN): now also R2.2
- net OSC_OUT: now reaches IC1.24 (OSC_OUT)
- net OSC_OUT: now also Y4.3
- net OSC_IN: now reaches IC1.25 (OSC_IN)
- net OSC_IN: now also Y4.1
- net AT0: now reaches IC1.26 (AT0)
- net AT0: now also J16.14 (Pin_14)
- net AT1: now reaches IC1.27 (AT1)
- net AT1: now also J16.13 (Pin_13)
- net PA10_USART1_RX: now reaches IC1.36 (PA10)
- net PA10_USART1_RX: now also J15.4 (Pin_4)
- net PA11_USB_D-: now reaches IC1.37 (PA11)
- net PA12_USB_D+: now reaches IC1.38 (PA12)
- net PA13_SWDIO: now reaches IC1.39 (PA13)
- net PA14_SWCLK: now reaches IC1.41 (PA14)
- net PB3_SWO: now reaches IC1.43 (PB3)
- net PB4_I2C3_SDA: now reaches IC1.44 (PB4)
- net PB4_I2C3_SDA: now also J7.4 (Pin_4)
- net PB5_SPI1_MOSI: now reaches IC1.45 (PB5)
- net PB5_SPI1_MOSI: now also J20.5 (Pin_5)
- net PB6: now reaches IC1.46 (PB6)
- net PB6: now also J16.8 (Pin_8)
- net PB7: now reaches IC1.47 (PB7)
- net PB7: now also J16.7 (Pin_7)
- new net: R2.1, Y3.3 (OUTPUT)
- new net: BH1.1 (+), J4.3 (Pin_3)
Other:
- note added: "Average Current 8.8 mA (Estimated from report) 1. Programming - SW is inteneded but all pins will be exposed for possible JTAG interface 2. LDO is intended to be used with USB VBUS power supply (When running the device through USB power) 4u7F Capacitor Placement Strategy: Near the Most Critical VDD Pin If one VDD pin powers the core logic (e.g., MCU core supply), place the 4.7µF capacitor closest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"
- note added: "EP is optional adhesive zone"
- note added: "On UFQFPN48 VDDA is connected to VREF+."
- note removed: "1. Programming - SW is inteneded but all pins will be exposed for possible JTAG interface 2. LDO is intended to be used with USB VBUS power supply (When running the device through USB power) Approximate Current Consumption (at 3.3V VDD) Run Mode (CPU active at 64 MHz): Typ: ~9.2 mA Max: ~14.4 mA Sleep Mode (CPU stopped, peripherals active): Typ: ~4.8 mA Stop Mode (Low-power mode with retention, 3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"
- note removed: "100 nF for each VDD or VDDIO2 (Ceramic capacitors) Place very close"
- note removed: "FT 5 V tolerant I/O"
- note removed: "PWR_FLG tells KiCad that this is power source"
- moved on the sheet: C12, C24, C25, C7, C9, ESD1, ESD2, FLT1, H1, H2, H3, H4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

Commit message: Update
Parts:
- removed J16: Pin_Header, Connector_PinHeader_2.54mm:PinHeader_2x07_P2.54mm_Vertical, symbol Connector_Generic:Conn_02x07_Odd_Even
- added J12: Pin_Header, Connector_PinHeader_2.54mm:PinHeader_2x06_P2.54mm_Vertical, symbol Connector_Generic:Conn_02x06_Odd_Even
- C19, C20, C21, C22, C23, C24, C25, C26, C27, C28, C29, C30, C31, C32, C33, C34, C35, C36, C9: footprint Capacitor_SMD:C_0805_2012Metric_Pad1.18x1.45mm_HandSolder -> Capacitor_SMD:C_0603_1608Metric_Pad1.08x0.95mm_HandSolder
- J14: footprint Connector_PinSocket_2.54mm:PinSocket_2x04_P2.54mm_Vertical -> Connector_PinHeader_2.54mm:PinHeader_2x04_P2.54mm_Vertical
Connections:
- net GND: now also J12.1 (Pin_1)
- net PA0: now also J12.5 (Pin_5)
- net PA15: now also J12.9 (Pin_9)
- net PA5: now also J12.4 (Pin_4)
- net PA8_MCO: now also J12.3 (Pin_3)
- net PB0: now also J12.12 (Pin_12)
- net PB1: now also J12.11 (Pin_11)
- net PB2: now also J12.2 (Pin_2)
- net PB6: now also J12.8 (Pin_8)
- net PB7: now also J12.7 (Pin_7)
- net PC15-OSC32_OUT: now also J12.6 (Pin_6)
- net PE4: now also J12.10 (Pin_10)
- net AT0: no longer names the net of IC1.26 (AT0)
- net AT1: no longer names the net of IC1.27 (AT1)
- no-connect marks 4 -> 6
Changed lines of the file:
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@@
 	)
 	(no_connect
+		(at 107.95 144.78)
+	)
+	(no_connect
 		(at 67.31 307.34)
 	)
@@
 	)
 	(no_connect
+		(at 107.95 142.24)
+	)
+	(no_connect
 		(at 227.33 124.46)
 	)
@@
 	(wire
 		(pts
-			(xy 401.32 240.03) (xy 425.45 240.03)
-		)
-		(stroke
-			(width 0)
-			(type default)
-		)
-	)
-	(wire
-		(pts
 			(xy 394.97 60.96) (xy 394.97 63.5)
 		)
@@
 	(wire
 		(pts
-			(xy 388.62 240.03) (xy 367.03 240.03)
-		)
-		(stroke
-			(width 0)
-			(type default)
-		)
-	)
-	(wire
-		(pts
 			(xy 210.82 317.5) (xy 210.82 306.07)
 		)
@@
 	(wire
 		(pts
-			(xy 92.71 144.78) (xy 107.95 144.78)
-		)
-		(stroke
-			(width 0)
-			(type default)
-		)
-	)
-	(wire
-		(pts
 			(xy 182.88 85.09) (xy 182.88 87.63)
 		)
@@
 	(wire
 		(pts
-			(xy 92.71 142.24) (xy 107.95 142.24)
-		)
-		(stroke
-			(width 0)
-			(type default)
-		)
-	)
-	(wire
-		(pts
 			(xy 393.7 304.8) (xy 393.7 302.26)
 		)
@@
 		)
 	)
-	(label "AT1"
-		(at 370.84 240.03 180)
-		(fields_autoplaced yes)
-		(effects
-			(font
-				(size 1.27 1.27)
-			)
-			(justify right bottom)
-		)
-	)
 	(label "PA11_USB_D-"
 		(at 495.3 55.88 180)
@@
 		)
 	)
-	(label "AT0"
-		(at 425.45 240.03 180)
-		(fields_autoplaced yes)
-		(effects
-			(font
-				(size 1.27 1.27)
-			)
-			(justify right bottom)
-		)
-	)
 	(label "PB3_SWO"
 		(at 525.78 116.84 0)
@@
 		)
 	)
-	(label "AT1"
-		(at 96.52 142.24 180)
-		(fields_autoplaced yes)
-		(effects
-			(font
-				(size 1.27 1.27)
-			)
-			(justify right bottom)
-		)
-	)
 	(label "RF_ANT"
 		(at 360.68 50.8 180)
@@
 		)
 	)
-	(label "AT0"
-		(at 96.52 144.78 180)
-		(fields_autoplaced yes)
-		(effects
-			(font
-				(size 1.27 1.27)
-			)
-			(justify right bottom)
-		)
-	)
 	(symbol
 		(lib_id "Device:C")
@@
 			)
 		)
-		(property "Footprint" "Capacitor_SMD:C_0805_2012Metric_Pad1.18x1.45mm_HandSolder"
+		(property "Footprint" "Capacitor_SMD:C_0603_1608Metric_Pad1.08x0.95mm_HandSolder"
 			(at 113.9952 204.47 0)
 			(effects
@@
 			)
 		)
-		(property "Footprint" "Capacitor_SMD:C_0805_2012Metric_Pad1.18x1.45mm_HandSolder"
+		(property "Footprint" "Capacitor_SMD:C_0603_1608Metric_Pad1.08x0.95mm_HandSolder"
 			(at 55.5752 153.67 0)
 			(effects
@@
 			)
 		)
-		(property "Footprint" "Capacitor_SMD:C_0805_2012Metric_Pad1.18x1.45mm_HandSolder"
+		(property "Footprint" "Capacitor_SMD:C_0603_1608Metric_Pad1.08x0.95mm_HandSolder"
 			(at 192.0748 198.12 0)
 			(effects
@@
 			)
 		)
-		(property "Footprint" "Capacitor_SMD:C_0805_2012Metric_Pad1.18x1.45mm_HandSolder"
+		(property "Footprint" "Capacitor_SMD:C_0603_1608Metric_Pad1.08x0.95mm_HandSolder"
 			(at 112.0648 184.15 0)
 			(effects
@@
 			)
 		)
-		(property "Footprint" "Capacitor_SMD:C_0805_2012Metric_Pad1.18x1.45mm_HandSolder"
+		(property "Footprint" "Capacitor_SMD:C_0603_1608Metric_Pad1.08x0.95mm_HandSolder"
 			(at 141.9352 377.19 0)
 			(effects
@@
 			)
 		)
-		(property "Footprint" "Connector_PinSocket_2.54mm:PinSocket_2x04_P2.54mm_Vertical"
+		(property "Footprint" "Connector_PinHeader_2.54mm:PinHeader_2x04_P2.54mm_Vertical"
 			(at 515.62 114.3 0)
 			(effects
@@
 			)
 		)
-		(property "Footprint" "Capacitor_SMD:C_0805_2012Metric_Pad1.18x1.45mm_HandSolder"
+		(property "Footprint" "Capacitor_SMD:C_0603_1608Metric_Pad1.08x0.95mm_HandSolder"
 			(at 116.5352 309.88 0)
 			(effects
@@
 			)
 		)
-		(property "Footprint" "Capacitor_SMD:C_0805_2012Metric_Pad1.18x1.45mm_HandSolder"
+		(property "Footprint" "Capacitor_SMD:C_0603_1608Metric_Pad1.08x0.95mm_HandSolder"
 			(at 362.9152 113.03 0)
 			(effects
@@
 			)
 		)
-		(property "Footprint" "Capacitor_SMD:C_0805_2012Metric_Pad1.18x1.45mm_HandSolder"
+		(property "Footprint" "Capacitor_SMD:C_0603_1608Metric_Pad1.08x0.95mm_HandSolder"
 			(at 131.7752 83.82 0)
 			(effects
@@
 			)
 		)
-		(property "Footprint" "Capacitor_SMD:C_0805_2012Metric_Pad1.18x1.45mm_HandSolder"
+		(property "Footprint" "Capacitor_SMD:C_0603_1608Metric_Pad1.08x0.95mm_HandSolder"
 			(at 204.7748 198.12 0)
 			(effects
@@
 			)
 		)
-		(property "Footprint" "Capacitor_SMD:C_0805_2012Metric_Pad1.18x1.45mm_HandSolder"
+		(property "Footprint" "Capacitor_SMD:C_0603_1608Metric_Pad1.08x0.95mm_HandSolder"
 			(at 183.8452 378.46 0)
 			(effects
@@
 			)
 		)
-		(property "Footprint" "Capacitor_SMD:C_0805_2012Metric_Pad1.18x1.45mm_HandSolder"
+		(property "Footprint" "Capacitor_SMD:C_0603_1608Metric_Pad1.08x0.95mm_HandSolder"
 			(at 203.2 131.7752 0)
 			(effects
@@
 			)
 		)
-		(property "Footprint" "Capacitor_SMD:C_0805_2012Metric_Pad1.18x1.45mm_HandSolder"
+		(property "Footprint" "Capacitor_SMD:C_0603_1608Metric_Pad1.08x0.95mm_HandSolder"
 			(at 56.1848 111.76 0)
 			(effects
@@
 			)
 		)
-		(property "Footprint" "Capacitor_SMD:C_0805_2012Metric_Pad1.18x1.45mm_HandSolder"
+		(property "Footprint" "Capacitor_SMD:C_0603_1608Metric_Pad1.08x0.95mm_HandSolder"
 			(at 159.7152 101.6 0)
 			(effects
@@
 			)
 		)
-		(property "Footprint" "Capacitor_SMD:C_0805_2012Metric_Pad1.18x1.45mm_HandSolder"
+		(property "Footprint" "Capacitor_SMD:C_0603_1608Metric_Pad1.08x0.95mm_HandSolder"
 			(at 85.3948 113.03 0)
 			(effects
@@
 	)
 	(symbol
-		(lib_id "Connector_Generic:Conn_02x07_Odd_Even")
-		(at 393.7 232.41 0)
-		(unit 1)
-		(exclude_from_sim no)
-		(in_bom yes)
-		(on_board yes)
-		(dnp no)
-		(property "Reference" "J16"
-			(at 395.224 220.98 0)
-			(effects
-				(font
-					(size 1.27 1.27)
-				)
-			)
-		)
-		(property "Value" "Pin_Header"
-			(at 394.97 243.332 0)
-			(effects
-				(font
-					(size 1.27 1.27)
-				)
-			)
-		)
-		(property "Footprint" "Connector_PinHeader_2.54mm:PinHeader_2x07_P2.54mm_Vertical"
-			(at 393.7 232.41 0)
-			(effects
-				(font
-					(size 1.27 1.27)
-				)
-				(hide yes)
-			)
-		)
-		(property "Datasheet" "~"
-			(at 393.7 232.41 0)
-			(effects
-				(font
-					(size 1.27 1.27)
-				)
-				(hide yes)
-			)
-		)
-		(property "Description" "Generic connector, double row, 02x07, odd/even pin numbering scheme (row 1 odd numbers, row 2 even numbers), script generated (kicad-library-utils/schlib/autogen/connector/)"
-			(at 393.7 232.41 0)
-			(effects
-				(font
-					(size 1.27 1.27)
-				)
-				(hide yes)
-			)
-		)
-		(pin "12"
-		)
-		(pin "10"
-		)
-		(pin "11"
-		)
-		(pin "1"
-		)
-		(pin "13"
-		)
-		(pin "14"
-		)
-		(pin "2"
-		)
-		(pin "3"
-		)
-		(pin "4"
-		)
-		(pin "5"
-		)
-		(pin "6"
-		)
-		(pin "7"
-		)
-		(pin "8"
-		)
-		(pin "9"
-		)
-		(instances
-			(project ""
-				(path "/05989bb3-969e-4aaa-b344-5f0e2d5af968"
-					(reference "J16")
-					(unit 1)
-				)
-			)
-		)
-	)
-	(symbol
 		(lib_id "Personal_Projects:DLF162500LT-5028A1")
 		(at 373.38 50.8 0)
@@
 			)
 		)
-		(property "Footprint" "Capacitor_SMD:C_0805_2012Metric_Pad1.18x1.45mm_HandSolder"
+		(property "Footprint" "Capacitor_SMD:C_0603_1608Metric_Pad1.08x0.95mm_HandSolder"
 			(at 206.7052 160.02 0)
 			(effects
@@
 			)
 		)
-		(property "Footprint" "Capacitor_SMD:C_0805_2012Metric_Pad1.18x1.45mm_HandSolder"
+		(property "Footprint" "Capacitor_SMD:C_0603_1608Metric_Pad1.08x0.95mm_HandSolder"
 			(at 99.3648 184.15 0)
 			(effects
@@
 			)
 		)
-		(property "Footprint" "Capacitor_SMD:C_0805_2012Metric_Pad1.18x1.45mm_HandSolder"
+		(property "Footprint" "Capacitor_SMD:C_0603_1608Metric_Pad1.08x0.95mm_HandSolder"
 			(at 72.6948 113.03 0)
 			(effects
@@
 			)
 		)
-		(property "Footprint" "Capacitor_SMD:C_0805_2012Metric_Pad1.18x1.45mm_HandSolder"
+		(property "Footprint" "Capacitor_SMD:C_0603_1608Metric_Pad1.08x0.95mm_HandSolder"
 			(at 183.8452 95.25 0)
 			(effects
@@
 			)
 		)
-		(property "Footprint" "Capacitor_SMD:C_0805_2012Metric_Pad1.18x1.45mm_HandSolder"
+		(property "Footprint" "Capacitor_SMD:C_0603_1608Metric_Pad1.08x0.95mm_HandSolder"
 			(at 247.3452 313.69 0)
 			(effects
@@
 					(unit 1)
 				)
+			)
+		)
+	)
+	(symbol
+		(lib_id "Connector_Generic:Conn_02x06_Odd_Even")
+		(at 393.7 229.87 0)
+		(unit 1)
+		(exclude_from_sim no)
+		(in_bom yes)
+		(on_board yes)
+		(dnp no)
+		(property "Reference" "J12"
+			(at 394.716 221.488 0)
+			(effects
+				(font
+					(size 1.27 1.27)
+				)
+			)
+		)
+		(property "Value" "Pin_Header"
+			(at 395.478 240.792 0)
+			(effects
+				(font
+					(size 1.27 1.27)
+				)
+			)
+		)
+		(property "Footprint" "Connector_PinHeader_2.54mm:PinHeader_2x06_P2.54mm_Vertical"
+			(at 393.7 229.87 0)
+			(effects
+				(font
+					(size 1.27 1.27)
+				)
+				(hide yes)
+			)
+		)
+		(property "Datasheet" "~"
+			(at 393.7 229.87 0)
+			(effects
+				(font
+					(size 1.27 1.27)
+				)
+				(hide yes)
+			)
+		)
+		(property "Description" "Generic connector, double row, 02x06, odd/even pin numbering scheme (row 1 odd numbers, row 2 even numbers), script generated (kicad-library-utils/schlib/autogen/connector/)"
+			(at 393.7 229.87 0)
+			(effects
+				(font
+					(size 1.27 1.27)
+				)
+				(hide yes)
+			)
+		)
+		(pin "3"
+		)
+		(pin "8"
+		)
+		(pin "10"
+		)
+		(pin "6"
+		)
+		(pin "1"
+		)
+		(pin "12"
+		)
+		(pin "4"
+		)
+		(pin "2"
+		)
+		(pin "9"
+		)
+		(pin "5"
+		)
+		(pin "7"
+		)
+		(pin "11"
+		)
+		(instances
+			(project ""
+				(path "/05989bb3-969e-4aaa-b344-5f0e2d5af968"
+					(reference "J12")
+					(unit 1)
+				)

Commit message: Update
Parts:
- removed J12: Pin_Header, Connector_PinHeader_2.54mm:PinHeader_2x06_P2.54mm_Vertical, symbol Connector_Generic:Conn_02x06_Odd_Even
- removed J7: I2C3_Header, Connector_PinHeader_2.54mm:PinHeader_1x04_P2.54mm_Vertical, symbol Connector_Generic:Conn_01x04
- added J7: Pin_Header, Connector_PinHeader_2.54mm:PinHeader_2x07_P2.54mm_Vertical, symbol Connector_Generic:Conn_02x07_Odd_Even
- R2, R6: footprint Resistor_SMD:R_0805_2012Metric_Pad1.20x1.40mm_HandSolder -> Resistor_SMD:R_0603_1608Metric_Pad0.98x0.95mm_HandSolder
Connections:
- net GND: now also J7.2 (Pin_2)
- net PA0: now also J7.5 (Pin_5)
- net PA15: now also J7.9 (Pin_9)
- net PA8_MCO: now also J7.3 (Pin_3)
- net PB0: now also J7.13 (Pin_13)
- net PB1: now also J7.14 (Pin_14)
- net PB2: now also J7.1 (Pin_1)
- net PC15-OSC32_OUT: now also J7.8 (Pin_8); no longer IC1.3 (PC15-OSC32_OUT)
- net PE4: now also J7.11 (Pin_11)
- net PA10_USART1_RX renamed PA10
- net PA10: now also J7.12 (Pin_12); no longer J15.4 (Pin_4)
- net PA1_SPI1_SCK renamed PA1
- net PA1: now also J7.6 (Pin_6); no longer J20.3 (Pin_3)
- net PA5 renamed PA5_SPI1_SCK
- net PA5_SPI1_SCK: now also J20.5 (Pin_5)
- net PA7_I2C3_SCL renamed PA7_SPI1_MOSI
- net PA7_SPI1_MOSI: now also J20.3 (Pin_3)
- net PA9_USART1_TX renamed PA9
- net PA9: now also J7.4 (Pin_4); no longer J15.3 (Pin_3)
- net PB4_I2C3_SDA renamed PB4
- net PB4: now also J7.10 (Pin_10)
- net PB5_SPI1_MOSI renamed PB5
- net PB5: now also J7.7 (Pin_7); no longer J20.5 (Pin_5)
- net PB6 renamed PB6_USART1_TX
- net PB6_USART1_TX: now also J15.3 (Pin_3)
- net PB7 renamed PB7_USART1_RX
- net PB7_USART1_RX: now also J15.4 (Pin_4)
- no-connect marks 6 -> 7
