File: Bluetooth_Board.kicad_sch (KiCad schematic)
At the start: 61 parts, among them IC1 STM32WB55CGU6, J1 5V Power Pins, J10 LPUART1_Header, J11 3V3 Power Pins, J13 3V3 Power Source Jumpers, J14 Debug_Pins, J15 USART1_Header, J19 Power Select Jumpers, J2 SMA PCB END LAUNCH JACK ROUND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, J20 SPI1_Header, J3 User Button Jumper, J4 Coin Battery Jumper, J5 Power Pins, J6 USB_B_Micro, J7 Pin_Header, J8 BOOT0_Jumper, J9 I2C1_Header, U3 USBLC6-2SC6, Y3 Clock_ECS-327MVATX-7-CN-TR, Y4 ABM3B-32.000MHZ-8-R30-B1U-T

Commit message: Update
Connections:
- net PC15-OSC32_OUT is gone; now on net GND: J7.8 (Pin_8)
- net 5V_SW: now also ESD1.1 (I/O1); no longer ESD1.3 (I/O2)
Changed lines of the file:
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@@
 	)
 	(junction
+		(at 67.31 313.69)
+		(diameter 0)
+		(color 0 0 0 0)
+	)
+	(junction
 		(at 375.92 125.73)
 		(diameter 0)
@@
 	)
 	(junction
-		(at 72.39 313.69)
-		(diameter 0)
-		(color 0 0 0 0)
-	)
-	(junction
 		(at 213.36 172.72)
 		(diameter 0)
@@
 	)
 	(no_connect
-		(at 107.95 144.78)
+		(at 72.39 307.34)
 	)
 	(no_connect
-		(at 67.31 307.34)
+		(at 107.95 144.78)
 	)
 	(no_connect
@@
 	(wire
 		(pts
-			(xy 60.96 313.69) (xy 72.39 313.69)
+			(xy 60.96 313.69) (xy 67.31 313.69)
 		)
 		(stroke
@@
 	(wire
 		(pts
-			(xy 369.57 116.84) (xy 369.57 125.73)
+			(xy 67.31 313.69) (xy 78.74 313.69)
 		)
 		(stroke
@@
 	(wire
 		(pts
-			(xy 373.38 304.8) (xy 377.19 304.8)
+			(xy 369.57 116.84) (xy 369.57 125.73)
 		)
 		(stroke
@@
 	(wire
 		(pts
-			(xy 326.39 209.55) (xy 304.8 209.55)
+			(xy 373.38 304.8) (xy 377.19 304.8)
 		)
 		(stroke
@@
 	(wire
 		(pts
-			(xy 154.94 370.84) (xy 152.4 370.84)
+			(xy 326.39 209.55) (xy 304.8 209.55)
 		)
 		(stroke
@@
 	(wire
 		(pts
-			(xy 97.79 101.6) (xy 97.79 121.92)
+			(xy 154.94 370.84) (xy 152.4 370.84)
 		)
 		(stroke
@@
 	(wire
 		(pts
-			(xy 194.31 87.63) (xy 191.77 87.63)
+			(xy 97.79 101.6) (xy 97.79 121.92)
 		)
 		(stroke
@@
 	(wire
 		(pts
-			(xy 199.39 294.64) (xy 210.82 294.64)
+			(xy 194.31 87.63) (xy 191.77 87.63)
 		)
 		(stroke
@@
 	(wire
 		(pts
-			(xy 72.39 307.34) (xy 72.39 313.69)
+			(xy 199.39 294.64) (xy 210.82 294.64)
 		)
 		(stroke
@@
 	(wire
 		(pts
-			(xy 72.39 313.69) (xy 78.74 313.69)
-		)
-		(stroke
-			(width 0)
-			(type default)
-		)
-	)
-	(wire
-		(pts
 			(xy 204.47 292.1) (xy 213.36 292.1)
 		)
@@
 	(wire
 		(pts
+			(xy 67.31 307.34) (xy 67.31 313.69)
+		)
+		(stroke
+			(width 0)
+			(type default)
+		)
+	)
+	(wire
+		(pts
 			(xy 431.8 304.8) (xy 431.8 302.26)
 		)
@@
 	(label "PB5"
 		(at 133.35 95.25 90)
+		(fields_autoplaced yes)
 		(effects
 			(font
@@
 	(label "PA1"
 		(at 165.1 142.24 0)
+		(fields_autoplaced yes)
 		(effects
 			(font
@@
 	(label "PA10"
 		(at 100.33 119.38 0)
+		(fields_autoplaced yes)
 		(effects
 			(font
@@
 		)
 	)
-	(label "PC15-OSC32_OUT"
-		(at 429.26 236.22 180)
-		(fields_autoplaced yes)
-		(effects
-			(font
-				(size 1.27 1.27)
-			)
-			(justify right bottom)
-		)
-	)
 	(label "PB3_SWO"
 		(at 525.78 116.84 0)
@@
 	(label "PA9"
 		(at 130.81 180.34 270)
+		(fields_autoplaced yes)
 		(effects
 			(font
@@
 	(label "PB4"
 		(at 130.81 95.25 90)
+		(fields_autoplaced yes)
 		(effects
 			(font
@@
 					(unit 1)
 				)
+			)
+		)
+	)
+	(symbol
+		(lib_id "power:GND")
+		(at 429.26 236.22 90)
+		(unit 1)
+		(exclude_from_sim no)
+		(in_bom yes)
+		(on_board yes)
+		(dnp no)
+		(property "Reference" "#PWR01"
+			(at 435.61 236.22 0)
+			(effects
+				(font
+					(size 1.27 1.27)
+				)
+				(hide yes)
+			)
+		)
+		(property "Value" "GND"
+			(at 432.308 238.76 90)
+			(effects
+				(font
+					(size 1.27 1.27)
+				)
+				(justify left)
+				(hide yes)
+			)
+		)
+		(property "Footprint" ""
+			(at 429.26 236.22 0)
+			(effects
+				(font
+					(size 1.27 1.27)
+				)
+				(hide yes)
+			)
+		)
+		(property "Datasheet" ""
+			(at 429.26 236.22 0)
+			(effects
+				(font
+					(size 1.27 1.27)
+				)
+				(hide yes)
+			)
+		)
+		(property "Description" "Power symbol creates a global label with name \"GND\" , ground"
+			(at 429.26 236.22 0)
+			(effects
+				(font
+					(size 1.27 1.27)
+				)
+				(hide yes)
+			)
+		)
+		(pin "1"
+		)
+		(instances
+			(project "Bluetooth_Board"
+				(path "/05989bb3-969e-4aaa-b344-5f0e2d5af968"
+					(reference "#PWR01")
+					(unit 1)
+				)

Commit message: Update
Connections:
- net 3V3_SW: now also ESD2.1 (I/O1); no longer ESD2.3 (I/O2)
- net PA11_USB_D- renamed USB_D-
- net PA12_USB_D+ renamed USB_D+
Changed lines of the file:
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@@
 	)
 	(junction
-		(at 204.47 317.5)
-		(diameter 0)
-		(color 0 0 0 0)
-	)
-	(junction
 		(at 238.76 303.53)
 		(diameter 0)
@@
 	)
 	(junction
+		(at 199.39 317.5)
+		(diameter 0)
+		(color 0 0 0 0)
+	)
+	(junction
 		(at 86.36 104.14)
 		(diameter 0)
@@
 	)
 	(no_connect
-		(at 199.39 311.15)
+		(at 204.47 311.15)
 	)
 	(no_connect
@@
 	(wire
 		(pts
+			(xy 199.39 317.5) (xy 210.82 317.5)
+		)
+		(stroke
+			(width 0)
+			(type default)
+		)
+	)
+	(wire
+		(pts
 			(xy 236.22 306.07) (xy 238.76 306.07)
 		)
@@
 	(wire
 		(pts
-			(xy 193.04 317.5) (xy 204.47 317.5)
+			(xy 193.04 317.5) (xy 199.39 317.5)
 		)
 		(stroke
@@
 	(wire
 		(pts
-			(xy 204.47 311.15) (xy 204.47 317.5)
-		)
-		(stroke
-			(width 0)
-			(type default)
-		)
-	)
-	(wire
-		(pts
 			(xy 40.64 372.11) (xy 40.64 373.38)
 		)
@@
 	(wire
 		(pts
-			(xy 204.47 317.5) (xy 210.82 317.5)
+			(xy 199.39 311.15) (xy 199.39 317.5)
 		)
 		(stroke
@@
 		)
 	)
-	(text "Average Current 8.8 mA (Estimated from report)\n\n1. Programming - SW is inteneded but all pins will be exposed \nfor possible JTAG interface\n2. LDO is intended to be used with USB VBUS power supply\n   (When running the device through USB power)\n\n4u7F Capacitor Placement Strategy:\nNear the Most Critical VDD Pin\nIf one VDD pin powers the core logic (e.g., MCU core supply), place \nthe 4.7µF capacitor closest to that pin. This ensures stability where power \ndemand is highest. At a Central Power Distribution Point\nIf all VDD pins are connected to a common power plane, place the 4.7µF \ncapacitor near the entry point of VDD to the PCB or close to where power is \ndistributed to all VDD pins.\nThis helps smooth out power fluctuations before it reaches different ICs.\nComplement with Smaller Capacitors (0.1µF)\nPlace 0.1µF capacitors close to each VDD pin for high-frequency noise filtering.\nThe 4.7µF capacitor handles bulk power stabilization, while 0.1µF capacitors \nhandle high-frequency noise.\nGeneral Rule:\nIf in doubt, place the 4.7µF capacitor near the largest power consumer (MCU, RF module, etc.).\n\nUsing external oscilator as LSE the PC15-OSC32_OUT can be used as a GPIO\n\nVREF+ pin is not available on all packages, when not available it is internally bonded to\nVDDA. When the VREF+ is double-bonded with VDDA in a package, the internal\nvoltage reference buffer is not available and must be kept disabled (refer to the\ndatasheet for pinout descriptions).\n\nOn the STM32WB55CGU6, the AT0 (Alternate Test 0) pin is typically used for factory\ntesting and internal debugging by STMicroelectronics. It is not intended for user \napplications and generally should be left unconnected unless specified otherwise in \nthe reference manual or datasheet."
+	(text "Average Current 8.8 mA (Estimated from report)\n\n1. Programming - SW is inteneded but all pins will be exposed \nfor possible JTAG interface\n2. LDO is intended to be used with USB VBUS power supply\n   (When running the device through USB power)\n\n4u7F Capacitor Placement Strategy:\nNear the Most Critical VDD Pin\nIf one VDD pin powers the core logic (e.g., MCU core supply), place \nthe 4.7µF capacitor closest to that pin. This ensures stability where power \ndemand is highest. At a Central Power Distribution Point\nIf all VDD pins are connected to a common power plane, place the 4.7µF \ncapacitor near the entry point of VDD to the PCB or close to where power is \ndistributed to all VDD pins.\nThis helps smooth out power fluctuations before it reaches different ICs.\nComplement with Smaller Capacitors (0.1µF)\nPlace 0.1µF capacitors close to each VDD pin for high-frequency noise filtering.\nThe 4.7µF capacitor handles bulk power stabilization, while 0.1µF capacitors \nhandle high-frequency noise.\nGeneral Rule:\nIf in doubt, place the 4.7µF capacitor near the largest power consumer (MCU, RF module, etc.).\n\nUsing external oscilator as LSE the PC15-OSC32_OUT can be used as a GPIO\n\nVREF+ pin is not available on all packages, when not available it is internally bonded to\nVDDA. When the VREF+ is double-bonded with VDDA in a package, the internal\nvoltage reference buffer is not available and must be kept disabled (refer to the\ndatasheet for pinout descriptions).\n\nOn the STM32WB55CGU6, the AT0 (Alternate Test 0) pin is typically used for factory\ntesting and internal debugging by STMicroelectronics. It is not intended for user \napplications and generally should be left unconnected unless specified otherwise in \nthe reference manual or datasheet.\n\nUSB Differential Pair\nCalculated on JLCPB website\nbased on 90 Ohm, 0.25mm spacing, 9.35mm trace to copper\n0.1669 mmm track width"
 		(exclude_from_sim no)
-		(at 479.425 194.945 0)
+		(at 479.552 198.882 0)
 		(effects
 			(font
@@
 		)
 	)
-	(label "PA12_USB_D+"
-		(at 115.57 104.14 90)
+	(label "USB_D+"
+		(at 115.57 99.06 90)
+		(fields_autoplaced yes)
+		(effects
+			(font
+				(size 1.27 1.27)
+			)
+			(justify left bottom)
+		)
+	)
+	(label "USB_D+"
+		(at 481.33 53.34 0)
 		(fields_autoplaced yes)
 		(effects
@@
 		)
 	)
-	(label "PA11_USB_D-"
-		(at 495.3 55.88 180)
-		(fields_autoplaced yes)
-		(effects
-			(font
-				(size 1.27 1.27)
-			)
-			(justify right bottom)
-		)
-	)
 	(label "PB3_SWO"
 		(at 128.27 100.33 90)
@@
 		)
 	)
-	(label "PA12_USB_D+"
-		(at 495.3 53.34 180)
-		(fields_autoplaced yes)
-		(effects
-			(font
-				(size 1.27 1.27)
-			)
-			(justify right bottom)
-		)
-	)
 	(label "VBUS"
 		(at 45.72 297.18 0)
@@
 		)
 	)
+	(label "USB_D-"
+		(at 481.33 55.88 0)
+		(fields_autoplaced yes)
+		(effects
+			(font
+				(size 1.27 1.27)
+			)
+			(justify left bottom)
+		)
+	)
 	(label "PA13_SWDIO"
 		(at 118.11 102.87 90)
@@
 		)
 	)
-	(label "PA11_USB_D-"
-		(at 113.03 104.14 90)
+	(label "USB_D-"
+		(at 113.03 99.06 90)
 		(fields_autoplaced yes)
 		(effects
@@
 		(dnp no)
 		(property "Reference" "C36"
-			(at 203.962 161.798 0)
+			(at 203.454 161.544 0)
 			(effects
 				(font

Commit message: Update
Parts:
- removed H5: MountingHole_Pad, MountingHole:MountingHole_3.2mm_M3_Pad, symbol Mechanical:MountingHole_Pad
- J10: footprint Connector_PinHeader_2.54mm:PinHeader_1x04_P2.54mm_Vertical -> Connector_PinHeader_2.54mm:PinHeader_1x04_P2.54mm_Horizontal
- J20: footprint Connector_PinHeader_2.54mm:PinHeader_1x06_P2.54mm_Vertical -> Connector_PinHeader_2.54mm:PinHeader_1x06_P2.54mm_Horizontal
Connections:
- net +3.3V: now also J10.4 (Pin_4); no longer J10.1 (Pin_1)
- net GND: now also J10.3 (Pin_3); no longer J10.2 (Pin_2)
- net PA0: now also J7.4 (Pin_4); no longer J3.2 (Pin_2), J7.5 (Pin_5)
- net PA1: now also J3.2 (Pin_2), J7.1 (Pin_1); no longer J7.6 (Pin_6)
- net PA2_LPUART1_TX: now also J10.2 (Pin_2); no longer J10.3 (Pin_3)
- net PA3_LPUART1_RX: now also J10.1 (Pin_1); no longer J10.4 (Pin_4)
- net PA8_MCO: now also J7.5 (Pin_5); no longer J7.3 (Pin_3)
- net PA9: now also J7.6 (Pin_6); no longer J7.4 (Pin_4)
- net PB2: now also J7.3 (Pin_3); no longer J7.1 (Pin_1)
Other:
- moved on the sheet: H6

Commit message: Update
Parts:
- removed FB2: FCM1608KF-601T03, Inductor_SMD:L_0603_1608Metric_Pad1.05x0.95mm_HandSolder, symbol Device:FerriteBead
- added FB1: BLM21PG601SN1D_0805, Capacitor_SMD:C_0805_2012Metric_Pad1.18x1.45mm_HandSolder, symbol Device:FerriteBead
Connections:
- net +3.3V: now also FB1.2
- net +3.3VA: now also FB1.1
Changed lines of the file:
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@@
-	)
-	(symbol
-		(lib_id "Device:FerriteBead")
-		(at 213.36 189.23 270)
-		(mirror x)
-		(unit 1)
-		(exclude_from_sim no)
-		(in_bom yes)
-		(on_board yes)
-		(dnp no)
-		(property "Reference" "FB2"
-			(at 213.4108 181.61 90)
-			(effects
-				(font
-					(size 1.27 1.27)
-				)
-			)
-		)
-		(property "Value" "FCM1608KF-601T03"
-			(at 213.36 184.404 90)
-			(effects
-				(font
-					(size 1.27 1.27)
-				)
-			)
-		)
-		(property "Footprint" "Inductor_SMD:L_0603_1608Metric_Pad1.05x0.95mm_HandSolder"
-			(at 213.36 191.008 90)
-			(effects
-				(font
-					(size 1.27 1.27)
-				)
-				(hide yes)
-			)
-		)
-		(property "Datasheet" "~"
-			(at 213.36 189.23 0)
-			(effects
-				(font
-					(size 1.27 1.27)
-				)
-				(hide yes)
-			)
-		)
-		(property "Description" "Ferrite bead"
-			(at 213.36 189.23 0)
-			(effects
-				(font
-					(size 1.27 1.27)
-				)
-				(hide yes)
-			)
-		)
-		(pin "1"
-		)
-		(pin "2"
-		)
-		(instances
-			(project "Bluetooth_Board"
-				(path "/05989bb3-969e-4aaa-b344-5f0e2d5af968"
-					(reference "FB2")
-					(unit 1)
-				)
-			)
-		)
 	)
 	(symbol
@@
 					(unit 1)
 				)
+			)
+		)
+	)
+	(symbol
+		(lib_id "Device:FerriteBead")
+		(at 213.36 189.23 90)
+		(unit 1)
+		(exclude_from_sim no)
+		(in_bom yes)
+		(on_board yes)
+		(dnp no)
+		(property "Reference" "FB1"
+			(at 217.932 187.706 90)
+			(effects
+				(font
+					(size 1.27 1.27)
+				)
+			)
+		)
+		(property "Value" "BLM21PG601SN1D_0805"
+			(at 223.012 193.548 90)
+			(effects
+				(font
+					(size 1.27 1.27)
+				)
+			)
+		)
+		(property "Footprint" "Capacitor_SMD:C_0805_2012Metric_Pad1.18x1.45mm_HandSolder"
+			(at 213.36 191.008 90)
+			(effects
+				(font
+					(size 1.27 1.27)
+				)
+				(hide yes)
+			)
+		)
+		(property "Datasheet" "~"
+			(at 213.36 189.23 0)
+			(effects
+				(font
+					(size 1.27 1.27)
+				)
+				(hide yes)
+			)
+		)
+		(property "Description" "Ferrite bead"
+			(at 213.36 189.23 0)
+			(effects
+				(font
+					(size 1.27 1.27)
+				)
+				(hide yes)
+			)
+		)
+		(pin "1"
+		)
+		(pin "2"
+		)
+		(instances
+			(project "Bluetooth_Board"
+				(path "/05989bb3-969e-4aaa-b344-5f0e2d5af968"
+					(reference "FB1")
+					(unit 1)
+				)
