File: Bluetooth_Board.kicad_sch (KiCad schematic)
At the start: 60 parts, among them IC1 STM32WB55CGU6, J1 5V Power Pins, J10 LPUART1_Header, J11 3V3 Power Pins, J13 3V3 Power Source Jumpers, J14 Debug_Pins, J15 USART1_Header, J19 Power Select Jumpers, J2 SMA PCB END LAUNCH JACK ROUND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, J20 SPI1_Header, J3 User Button Jumper, J4 Coin Battery Jumper, J5 Power Pins, J6 USB_B_Micro, J7 Pin_Header, J8 BOOT0_Jumper, J9 I2C1_Header, U3 USBLC6-2SC6, Y3 Clock_ECS-327MVATX-7-CN-TR, Y4 ABM3B-32.000MHZ-8-R30-B1U-T

Commit message: Update
Parts:
- removed Y3: Clock_ECS-327MVATX-7-CN-TR, Personal_Project:Clock_ECS327MVATX7CNTR, symbol Personal_Projects:Clock_ECS-327MVATX-7-CN-TR
- added OS1: Oscillator_ECS-327MVATX-3-CN-TR, Personal_Project:Oscillator_ECS327MVATX3CNTR, symbol Personal_Projects:Oscillator_ECS-327MVATX-3-CN-TR
Connections:
- net +3.3V: now also OS1.4 (VDD)
- net GND: now also OS1.2 (GND)
- net at R2.1: now also OS1.3 (OUTPUT)
Other:
- note removed: "Average Current 8.8 mA (Estimated from report) 1. Programming - SW is inteneded but all pins will be exposed for possible JTAG interface 2. LDO is intended to be used with USB VBUS power supply (When running the device through USB power) 4u7F Capacitor Placement Strategy: Near the Most Critical VDD Pin If one VDD pin powers the core logic (e.g., MCU core supply), place the 4.7µF capacitor closest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"

Commit message: update
Parts:
- removed C23, C26: 4u7, Capacitor_SMD:C_0603_1608Metric_Pad1.08x0.95mm_HandSolder, symbol Device:C
- removed ESD1, ESD2: ESDALC6V1W5, Personal_Project:SOT323-5L_STM-L, symbol Personal_Projects:ESDALC6V1W5
- removed H6: MountingHole_Pad, MountingHole:MountingHole_3.2mm_M3_Pad, symbol Mechanical:MountingHole_Pad
- removed J10: LPUART1_Header, Connector_PinHeader_2.54mm:PinHeader_1x04_P2.54mm_Horizontal, symbol Connector_Generic:Conn_01x04
- removed J11: 3V3 Power Pins, Connector_PinHeader_2.54mm:PinHeader_2x03_P2.54mm_Vertical, symbol Connector_Generic:Conn_02x03_Odd_Even
- removed J13: 3V3 Power Source Jumpers, Personal_Project:PinHeader_2x03_P2.54mm_Vertical_PINS, symbol Connector_Generic:Conn_02x03_Top_Bottom
- removed J14: Debug_Pins, Connector_PinHeader_2.54mm:PinHeader_2x04_P2.54mm_Vertical, symbol Connector_Generic:Conn_02x04_Odd_Even
- removed J15: USART1_Header, Connector_PinHeader_2.54mm:PinHeader_1x04_P2.54mm_Vertical, symbol Connector_Generic:Conn_01x04
- removed J17: ~, Personal_Project:SMA Clip Mount Adapter (bottom), symbol Personal_Projects:SMA_PCB_END_JACK_(BOTTOM)
- removed J19: Power Select Jumpers, Personal_Project:PinHeader_2x03_P2.54mm_Vertical_PINS, symbol Connector_Generic:Conn_02x03_Top_Bottom
- removed J20: SPI1_Header, Connector_PinHeader_2.54mm:PinHeader_1x06_P2.54mm_Horizontal, symbol Connector_Generic:Conn_01x06
- removed J5: Power Pins, Connector_PinHeader_2.54mm:PinHeader_1x04_P2.54mm_Vertical, symbol Connector:Conn_01x04_Pin
- removed J6: USB_B_Micro, Connector_USB:USB_Micro-B_Molex-105017-0001, symbol Connector:USB_B_Micro
- removed J9: I2C1_Header, Connector_PinHeader_2.54mm:PinHeader_1x04_P2.54mm_Vertical, symbol Connector_Generic:Conn_01x04
- removed OS1: Oscillator_ECS-327MVATX-3-CN-TR, Personal_Project:Oscillator_ECS327MVATX3CNTR, symbol Personal_Projects:Oscillator_ECS-327MVATX-3-CN-TR
- added C2: 4u7, Capacitor_SMD:C_0805_2012Metric, symbol Device:C
- added D1: BZX84C4V3LT1G, Package_TO_SOT_SMD:SOT-23, symbol Diode:BZX84Cxx
- added D2: BZX84C6V2LT1G, Package_TO_SOT_SMD:SOT-23, symbol Diode:BZX84Cxx
- added J10: Debug_Pins, Connector_PinHeader_2.54mm:PinHeader_2x04_P2.54mm_Horizontal, symbol Connector_Generic:Conn_02x04_Odd_Even
- added J12: Power_Selector_Jumper, Connector_PinHeader_2.54mm:PinHeader_2x03_P2.54mm_Vertical, symbol Connector_Generic:Conn_02x03_Odd_Even
- added J13: General_Pin_Header, Connector_PinHeader_2.54mm:PinHeader_2x07_P2.54mm_Horizontal, symbol Connector_Generic:Conn_02x07_Odd_Even
- added J14: JST_XH_2.54_Plug, Personal_Project:Connector_Power2pin_SHDRRA2W80P0X250_1X2_740X1150X610P, symbol Personal_Projects:Connector_Power2pin_JST_XH_2.54_Plug
- added J15: LPUART1_Headers, Connector_PinHeader_2.54mm:PinHeader_2x03_P2.54mm_Horizontal, symbol Connector_Generic:Conn_02x03_Odd_Even
- added J16: SPI1_Headers, Connector_PinHeader_2.54mm:PinHeader_2x03_P2.54mm_Horizontal, symbol Connector_Generic:Conn_02x03_Odd_Even
- added J19: 3V_Selection_Header, Connector_PinHeader_2.54mm:PinHeader_1x03_P2.54mm_Vertical, symbol Connector_Generic:Conn_01x03
- added J5: USB_B_Micro, Connector_USB:USB_Micro-B_XKB_U254-051T-4BH83-F1S, symbol Connector:USB_B_Micro
- added J6: I2C1_Headers, Connector_PinHeader_2.54mm:PinHeader_2x03_P2.54mm_Horizontal, symbol Connector_Generic:Conn_02x03_Odd_Even
- added OS2: Oscillator_ECS-327MVATX-3-CN-TR, Personal_Project:Oscillator_ECS327MVATX3CNTR, symbol Personal_Projects:Oscillator_ECS-327MVATX-3-CN-TR
- added Q1: MOSFET_SI2333DDS-T1-BE3, Personal_Project:MOSFET_ SI2333DDS_SOT_DS-T1-BE3_VIS, symbol Personal_Projects:MOSFET_SI2333DDS-T1-BE3
- added R1, R10, R11, R12, R13, R14, R3: 33R, Resistor_SMD:R_0805_2012Metric, symbol Device:R
- added R20: 100k, Resistor_SMD:R_0805_2012Metric, symbol Device:R
- added S2: Switch_WS-SLSU SMT Mini Slide, Personal_Project:Switch_WS-SLSU SMT Mini Slide, symbol Personal_Projects:Switch_WS-SLSU SMT Mini Slide
- added Z1: Diode_BZX84C6V2-7-F, Personal_Project:Diode_BZX84C6V2_SOT96P240X110-3N, symbol Personal_Projects:Diode_BZX84C6V2-7-F
- C19, C20, C21, C22, C24, C25, C27, C28, C29, C30, C31, C32, C33, C34, C35, C36, C9: footprint Capacitor_SMD:C_0603_1608Metric_Pad1.08x0.95mm_HandSolder -> Capacitor_SMD:C_0805_2012Metric
- FB1: footprint Capacitor_SMD:C_0805_2012Metric_Pad1.18x1.45mm_HandSolder -> Capacitor_SMD:C_0805_2012Metric
- J1: value 5V Power Pins -> USART1_Headers; footprint Connector_PinHeader_2.54mm:PinHeader_2x03_P2.54mm_Vertical -> Connector_PinHeader_2.54mm:PinHeader_2x03_P2.54mm_Horizontal
- J7: value Pin_Header -> General_Pin_Header; footprint Connector_PinHeader_2.54mm:PinHeader_2x07_P2.54mm_Vertical -> Connector_PinHeader_2.54mm:PinHeader_2x07_P2.54mm_Horizontal
- R2, R6: footprint Resistor_SMD:R_0603_1608Metric_Pad0.98x0.95mm_HandSolder -> Resistor_SMD:R_0805_2012Metric
Connections:
- net +3.3V: now also OS2.4 (VDD), S2.3
- net GND: now also J1.3 (Pin_3), J7.10 (Pin_10), J7.12 (Pin_12), J7.14 (Pin_14), J7.4 (Pin_4), J7.6 (Pin_6), C2.2, D1.1 (A), D2.1 (A), J10.1 (Pin_1), J10.3 (Pin_3), J10.5 (Pin_5), J10.7 (Pin_7), J13.10 (Pin_10), J13.12 (Pin_12), J13.14 (Pin_14), J13.2 (Pin_2), J13.3 (Pin_3), J13.4 (Pin_4), J13.6 (Pin_6), J13.8 (Pin_8), J14.1 (POWER-), J15.2 (Pin_2), J15.3 (Pin_3), J15.4 (Pin_4), J15.6 (Pin_6), J16.2 (Pin_2), J16.6 (Pin_6), J5.5 (GND), J5.6 (Shield), J6.2 (Pin_2), J6.3 (Pin_3), J6.4 (Pin_4), J6.6 (Pin_6), OS2.2 (GND), R20.2
- net LD_OUT_3V3: now also J19.3 (Pin_3)
- net NRST: now also J10.6 (Pin_6)
- net PA0: now also J13.11 (Pin_11); no longer J7.4 (Pin_4)
- net PA1: now also J13.9 (Pin_9); no longer J3.2 (Pin_2), J7.1 (Pin_1)
- net PA10: now also J7.1 (Pin_1); no longer J7.12 (Pin_12)
- net PA13_SWDIO: now also J10.8 (Pin_8)
- net PA14_SWCLK: now also J10.2 (Pin_2)
- net PA15: now also J13.7 (Pin_7); no longer J7.9 (Pin_9)
- net PA2_LPUART1_TX: now also R10.2
- net PA3_LPUART1_RX: now also R11.1
- net PA4_SPI1_NSS: now also J13.13 (Pin_13)
- net PA5_SPI1_SCK: now also R13.1
- net PA6_SPI1_MISO: now also R12.1
- net PA7_SPI1_MOSI: now also R14.2
- net PA8_MCO: now also J7.9 (Pin_9); no longer J7.5 (Pin_5)
- net PA9: now also J7.11 (Pin_11); no longer J7.6 (Pin_6)
- net PB0: now also J7.7 (Pin_7); no longer J7.13 (Pin_13)
- net PB1: now also J7.5 (Pin_5); no longer J7.14 (Pin_14)
- net PB2: now also J7.13 (Pin_13); no longer J7.3 (Pin_3)
- net PB3_SWO: now also J10.4 (Pin_4)
- net PB4: now also J13.5 (Pin_5); no longer J7.10 (Pin_10)
- net PB5: now also J3.2 (Pin_2), J13.1 (Pin_1); no longer J7.7 (Pin_7)
- net PB6_USART1_TX: now also R1.2
- net PB7_USART1_RX: now also R3.1
- net PB8_I2C1_SCL: now also J6.5 (Pin_5)
- net PB9_I2C1_SDA: now also J6.1 (Pin_1)
- net PE4: now also J7.3 (Pin_3); no longer J7.11 (Pin_11)
- net USB_D2+: now also J5.3 (D+)
- net USB_D2-: now also J5.2 (D-)
- net at R6.2: now also J5.4 (ID)
- net at R2.1: now also OS2.3 (OUTPUT)
- net +5V renamed LDO_IN
- net LDO_IN: now also J12.4 (Pin_4), J12.6 (Pin_6); no longer J1.1 (Pin_1), J1.3 (Pin_3), J1.5 (Pin_5)
- net VBUS renamed VBUS_5V
- net VBUS_5V: now also D2.3 (K), J12.5 (Pin_5), J5.1 (VBUS)
- new net: J16.4 (Pin_4), R14.1
- new net: J16.5 (Pin_5), R13.2
- new net: J15.5 (Pin_5), R11.2
- new net: J16.1 (Pin_1), R12.2
- new net: J1.1 (Pin_1), R1.1
- new net: J1.5 (Pin_5), R3.2
- new net: J15.1 (Pin_1), R10.1
- new net EXT_POWER+: J14.2 (POWER+), Q1.3 (D)
- new net EXT_POWER+_NOLDO: J12.2 (Pin_2), J19.1 (Pin_1)
- new net EXT_POWER+_PP: D1.3 (K), J12.1 (Pin_1), J12.3 (Pin_3), Q1.2 (S), Z1.3 (K)
- new net MOSFET_GATE: Q1.1 (G), R20.1, Z1.1 (A)
- new net POWER_3V3: C2.1, J19.2 (Pin_2), S2.2
- no-connect marks 7 -> 10
Other:
- note added: "Chip Select pin on general pin header"
- note added: "Input voltage range: 1.45V to 5.5V"
- note added: "ON/OFF Switch"
- note added: "Overvoltage protection for the PMOSFET VGS (VGS max is 8V)"
- note added: "Polarity Protection"
- note added: "ST-LINK Connections: VCP_TX, SWCLK, SWDIO, VCP_RX, NRST"
- note added: "STM32MP157FAD1 TFBGA257 Pitch 0.5 2x STM32WB55CGU6 2x STM32WB5MMGH6TR STM32MP135DAF7 TFBGA320 Pitch 0.5 STM32H7S7L8H6H STSPIN958TR STM32H7S3I8T6 LSM6DSV16XTR ISM330BXTR STM32WL55CCU6 STM32WL55JCI6 2x AGVLB.25B.07.0060A Connector: I-PEX MHF® I (U.FL Compatible) GW.52.A153 2.4/5.8/7.1GHZ Hinged RP-SMA (M) Connector TI.96.A113 900-940MHZ Connector: SMA(M) CS5381K-KSZ IC 120DB 192KHZ MULTI-BIT ADC 2x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"
- note removed: "STM32MP157FAD1 2x STM32WB55CGU6 2x STM32WB5MMGH6TR STM32MP135DAF7 STM32H7S7L8H6H STSPIN958TR STM32H7S3I8T6 LSM6DSV16XTR ISM330BXTR STM32WL55CCU6 STM32WL55JCI6 2x"
- moved on the sheet: H1, H2, H3, H4, J7

Commit message: Update
Parts:
- removed BH1: Battery_Holder_1060TR, Personal_Project:Battery_Holder_1060TR, symbol Personal_Projects:Battery_Holder_1060TR
- removed C12: 0p8 GRM1555C1HR80BA01D, Capacitor_SMD:C_0402_1005Metric_Pad0.74x0.62mm_HandSolder, symbol Device:C
- removed C19: 10n, Capacitor_SMD:C_0805_2012Metric, symbol Device:C
- removed C2, C28, C31, C32: 4u7, Capacitor_SMD:C_0805_2012Metric, symbol Device:C
- removed C20, C21, C22, C27, C29, C30, C33, C34: 100n, Capacitor_SMD:C_0805_2012Metric, symbol Device:C
- removed C24, C25, C35: 1u, Capacitor_SMD:C_0805_2012Metric, symbol Device:C
- removed C36, C9: 1uF, Capacitor_SMD:C_0805_2012Metric, symbol Device:C
- removed C7: 0p3 GRM1555C1HR30WA01D, Capacitor_SMD:C_0402_1005Metric_Pad0.74x0.62mm_HandSolder, symbol Device:C
- removed D1: BZX84C4V3LT1G, Package_TO_SOT_SMD:SOT-23, symbol Diode:BZX84Cxx
- removed D2: BZX84C6V2LT1G, Package_TO_SOT_SMD:SOT-23, symbol Diode:BZX84Cxx
- removed FB1: BLM21PG601SN1D_0805, Capacitor_SMD:C_0805_2012Metric, symbol Device:FerriteBead
- removed FLT1: DLF162500LT-5028A1, Personal_Project:DLF162500LT-5028A1, symbol Personal_Projects:DLF162500LT-5028A1
- removed H1, H2, H3, H4: MountingHole_Pad, MountingHole:MountingHole_3.2mm_M3_Pad, symbol Mechanical:MountingHole_Pad
- removed IC1: STM32WB55CGU6, Personal_Project:STM32WB55CGU6_QFN50P700X700X60-49N-D, symbol Personal_Projects:STM32WB55CGU6
- removed J1: USART1_Headers, Connector_PinHeader_2.54mm:PinHeader_2x03_P2.54mm_Horizontal, symbol Connector_Generic:Conn_02x03_Odd_Even
- removed J10: Debug_Pins, Connector_PinHeader_2.54mm:PinHeader_2x04_P2.54mm_Horizontal, symbol Connector_Generic:Conn_02x04_Odd_Even
- removed J12: Power_Selector_Jumper, Connector_PinHeader_2.54mm:PinHeader_2x03_P2.54mm_Vertical, symbol Connector_Generic:Conn_02x03_Odd_Even
- removed J13, J7: General_Pin_Header, Connector_PinHeader_2.54mm:PinHeader_2x07_P2.54mm_Horizontal, symbol Connector_Generic:Conn_02x07_Odd_Even
- removed J14: JST_XH_2.54_Plug, Personal_Project:Connector_Power2pin_SHDRRA2W80P0X250_1X2_740X1150X610P, symbol Personal_Projects:Connector_Power2pin_JST_XH_2.54_Plug
- removed J15: LPUART1_Headers, Connector_PinHeader_2.54mm:PinHeader_2x03_P2.54mm_Horizontal, symbol Connector_Generic:Conn_02x03_Odd_Even
- removed J16: SPI1_Headers, Connector_PinHeader_2.54mm:PinHeader_2x03_P2.54mm_Horizontal, symbol Connector_Generic:Conn_02x03_Odd_Even
- removed J19: 3V_Selection_Header, Connector_PinHeader_2.54mm:PinHeader_1x03_P2.54mm_Vertical, symbol Connector_Generic:Conn_01x03
- removed J2: SMA PCB END LAUNCH JACK ROUND PO, Personal_Project:SMA Clip Mount Adapter (top), symbol Personal_Projects:SMA PCB END LAUNCH JACK ROUND PO
- removed J3: User Button Jumper, Connector_PinHeader_2.54mm:PinHeader_1x02_P2.54mm_Vertical, symbol Connector_Generic:Conn_01x02
- removed J4: Coin Battery Jumper, Connector_PinHeader_2.54mm:PinHeader_1x03_P2.54mm_Vertical, symbol Connector_Generic:Conn_01x03
- removed J5: USB_B_Micro, Connector_USB:USB_Micro-B_XKB_U254-051T-4BH83-F1S, symbol Connector:USB_B_Micro
- removed J6: I2C1_Headers, Connector_PinHeader_2.54mm:PinHeader_2x03_P2.54mm_Horizontal, symbol Connector_Generic:Conn_02x03_Odd_Even
- removed J8: BOOT0_Jumper, Connector_PinHeader_2.54mm:PinHeader_1x03_P2.54mm_Vertical, symbol Connector:Conn_01x03_Pin
- removed L1: 2n7 LQG15HS2N7S02, Inductor_SMD:L_0402_1005Metric_Pad0.77x0.64mm_HandSolder, symbol Device:L
- removed L4: 10u Murata LQM21FN100M70L, Inductor_SMD:L_0805_2012Metric_Pad1.15x1.40mm_HandSolder, symbol Device:L
- removed L5: 10n Murata LQG15WZ10NJ02D, Inductor_SMD:L_0402_1005Metric_Pad0.77x0.64mm_HandSolder, symbol Device:L
- removed LDO1: LDO_TLV75733PDBVR, Personal_Project:LDO_SOT95P280X145-5N, symbol Personal_Projects:LDO_TLV75733PDBVR
- removed OS2: Oscillator_ECS-327MVATX-3-CN-TR, Personal_Project:Oscillator_ECS327MVATX3CNTR, symbol Personal_Projects:Oscillator_ECS-327MVATX-3-CN-TR
- removed Q1: MOSFET_SI2333DDS-T1-BE3, Personal_Project:MOSFET_ SI2333DDS_SOT_DS-T1-BE3_VIS, symbol Personal_Projects:MOSFET_SI2333DDS-T1-BE3
- removed R1, R10, R11, R12, R13, R14, R3: 33R, Resistor_SMD:R_0805_2012Metric, symbol Device:R
- removed R2: 10R, Resistor_SMD:R_0805_2012Metric, symbol Device:R
- removed R20, R6: 100k, Resistor_SMD:R_0805_2012Metric, symbol Device:R
- removed S2: Switch_WS-SLSU SMT Mini Slide, Personal_Project:Switch_WS-SLSU SMT Mini Slide, symbol Personal_Projects:Switch_WS-SLSU SMT Mini Slide
- removed U2, U6: ~, Personal_Project:Button_KMR231GLFS, symbol Personal_Projects:Button_KMR231GLFS
- removed U3: USBLC6-2SC6, Package_TO_SOT_SMD:SOT-23-6, symbol Power_Protection:USBLC6-2SC6
- removed Y4: ABM3B-32.000MHZ-8-R30-B1U-T, Personal_Project:XTAL_ABM3B-32.000MHZ-10-R30-B1U-T, symbol Personal_Projects:ABM3B-32.000MHZ-10-R30-B1U-T
- removed Z1: Diode_BZX84C6V2-7-F, Personal_Project:Diode_BZX84C6V2_SOT96P240X110-3N, symbol Personal_Projects:Diode_BZX84C6V2-7-F
Connections:
- no-connect marks 10 -> 0
Other:
- added sheet Interfaces (Interfaces.kicad_sch)
- added sheet Power_Management (Power_Management.kicad_sch)
- added sheet STM32WB55CGU6 (STM32WB55CGU6.kicad_sch)
- note removed: "120ohm at 100MHz"
- note removed: "2.4 GHz band antenna"
- note removed: "BOOT0 Switch HIGH enables UART or I2C to allow programminng of the MCU"
- note removed: "Can be used as GPIO"
- note removed: "Chip Select pin on general pin header"
- note removed: "Cloock Output"
- note removed: "Decide onn user button location ---------------"
- note removed: "EP is optional adhesive zone"
- note removed: "Footprint: 0402"
- note removed: "If shutdown capability is not required, connect EN to IN."
- note removed: "Input voltage range: 1.45V to 5.5V"
- note removed: "Load Capacitors are inside the MCU Set RCC_HSECR register"
- note removed: "NRST has internal pull-up resistor -When button not pushed NRST is HIGH -Pushing the button causes current to flow and pulls NRST low"
- note removed: "ON/OFF Switch"
- note removed: "On UFQFPN48 VDDA is connected to VREF+."
- note removed: "Overvoltage protection for the PMOSFET VGS (VGS max is 8V)"
- note removed: "PIN1 NC = Oscillation"
- note removed: "Polarity Protection"
- note removed: "ST-LINK Connections: VCP_TX, SWCLK, SWDIO, VCP_RX, NRST"
- note removed: "STM32MP157FAD1 TFBGA257 Pitch 0.5 2x STM32WB55CGU6 2x STM32WB5MMGH6TR STM32MP135DAF7 TFBGA320 Pitch 0.5 STM32H7S7L8H6H STSPIN958TR STM32H7S3I8T6 LSM6DSV16XTR ISM330BXTR STM32WL55CCU6 STM32WL55JCI6 2x AGVLB.25B.07.0060A Connector: I-PEX MHF® I (U.FL Compatible) GW.52.A153 2.4/5.8/7.1GHZ Hinged RP-SMA (M) Connector TI.96.A113 900-940MHZ Connector: SMA(M) CS5381K-KSZ IC 120DB 192KHZ MULTI-BIT ADC 2x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"
- note removed: "The external capacitor on NRST must be placed as close as possible to the device."
- note removed: "The load capacitances are integrated on chip and can be tuned according to the selected crystal via an internal register. By default, the load capacitances are 8 pF for the NX2016 from NDK used on the boards. RCC clock HSE register (RCC_HSECR) Bits 13:8 HSETUNE[5:0]: HSE capacitor tuning Can be changed by software. Do not change when HSE is on. 0x00: minimum load capacitance 0x3F maximum load cap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"
- note removed: "VDDA feeds ADC and DAC pins, and it needs more filtering"

Commit message: Update
Other:
- added sheet RF, USB (RF.kicad_sch)
- sheet Interfaces ports: added I2C_SCL_HDR, I2C_SDA_HDR, I/O_HDR0, I/O_HDR1, I/O_HDR2, I/O_HDR3, I/O_HDR4, I/O_HDR5, I/O_HDR6, I/O_HDR7, NRST, QSPI_CLK, QSPI_CS0, QSPI_IO0, QSPI_IO1, QSPI_IO2, QSPI_IO3, SPI_CLK, SPI_CS, SPI_MISO, SPI_MOSI, SWCLK, SWDIO, SWO, UART1_TX/RX, USR_BTN; removed none
- sheet Power_Management ports: added *RST; removed none
- sheet STM32WB55CGU6 ports: added PA10_I2C1_SDA, PA2_QUADSPI_BK1_NCS, PA3_QUADSPI_CLK, PA6_QUADSPI_BK1_IO3, PA7_QUADSPI_BK1_IO2, PA9_I2C1_SCL, PB4_SPI1_MISO, PB5_SPI1_MOSI, PB7, PB8_QUADSPI_BK1_IO1, PB9_QUADSPI_BK1_IO0; removed PA10, PA2_LPUART1_TX, PA3_LPUART1_RX, PA6_SPI1_MISO, PA7_SPI1_MOSI, PA9, PB4, PB5, PB7_USART1_RX, PB8_I2C1_SCL, PB9_I2C1_SDA

Commit message: Update
Other:
- sheet RF, USB ports: added USB_DI_D2+, USB_DI_D2-; removed USB_D2+_DI, USB_D2-_DI
Changed lines of the file:
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@@
 			)
 		)
-		(pin "USB_D2+_DI" bidirectional
+		(pin "USB_DI_D2+" bidirectional
 			(at 81.28 60.96 0)
 			(effects
@@
 			)
 		)
-		(pin "USB_D2-_DI" bidirectional
+		(pin "USB_DI_D2-" bidirectional
 			(at 81.28 63.5 0)
 			(effects

Commit message: Update
Connections:
- no-connect marks 0 -> 3
Other:
- sheet Interfaces ports: added none; removed I/O_HDR5, I/O_HDR6, I/O_HDR7, QSPI_CLK, QSPI_CS0, QSPI_IO0, QSPI_IO1, QSPI_IO2, QSPI_IO3
- sheet STM32WB55CGU6 ports: added none; removed PA2_QUADSPI_BK1_NCS, PA3_QUADSPI_CLK, PA6_QUADSPI_BK1_IO3, PA7_QUADSPI_BK1_IO2, PB8_QUADSPI_BK1_IO1, PB9_QUADSPI_BK1_IO0
