File: Interfaces.kicad_sch (KiCad schematic)
At the start: 27 parts, among them J12 SPI1_Headers, J14 SMA PCB END LAUNCH JACK ROUND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, J18 User Button Jumper, J19 LPUART1_Headers, J20 USART1_Headers, J21 General_Pin_Header, J22 General_Pin_Header, J23 I2C1_Headers, J24 Debug_Pins

Commit message: Update
Parts:
- removed C22: 0p3 GRM1555C1HR30WA01D, Capacitor_SMD:C_0402_1005Metric_Pad0.74x0.62mm_HandSolder, symbol Device:C
- removed C23: 0p8 GRM1555C1HR80BA01D, Capacitor_SMD:C_0402_1005Metric_Pad0.74x0.62mm_HandSolder, symbol Device:C
- removed DI2: Diode_PESD5V0U2BT-Q, Package_TO_SOT_SMD:SOT-23, symbol Personal_Projects:Diode_PESD5V0U2BT-Q
- removed FLT2: DLF162500LT-5028A1, Personal_Project:DLF162500LT-5028A1, symbol Personal_Projects:DLF162500LT-5028A1
- removed H5, H6, H7, H8: MountingHole_Pad, MountingHole:MountingHole_3.2mm_M3_Pad, symbol Mechanical:MountingHole_Pad
- removed J12: SPI1_Headers, Connector_PinHeader_2.54mm:PinHeader_2x03_P2.54mm_Horizontal, symbol Connector_Generic:Conn_02x03_Odd_Even
- removed J14: SMA PCB END LAUNCH JACK ROUND PO, Personal_Project:SMA Clip Mount Adapter (top), symbol Personal_Projects:SMA PCB END LAUNCH JACK ROUND PO
- removed J19: LPUART1_Headers, Connector_PinHeader_2.54mm:PinHeader_2x03_P2.54mm_Horizontal, symbol Connector_Generic:Conn_02x03_Odd_Even
- removed J20: USART1_Headers, Connector_PinHeader_2.54mm:PinHeader_2x03_P2.54mm_Horizontal, symbol Connector_Generic:Conn_02x03_Odd_Even
- removed J21, J22: General_Pin_Header, Connector_PinHeader_2.54mm:PinHeader_2x07_P2.54mm_Horizontal, symbol Connector_Generic:Conn_02x07_Odd_Even
- removed J23: I2C1_Headers, Connector_PinHeader_2.54mm:PinHeader_2x03_P2.54mm_Horizontal, symbol Connector_Generic:Conn_02x03_Odd_Even
- removed L4: 2n7 LQG15HS2N7S02, Inductor_SMD:L_0402_1005Metric_Pad0.77x0.64mm_HandSolder, symbol Device:L
- removed R15, R16, R17, R7, R8, R9: 33R, Resistor_SMD:R_0805_2012Metric, symbol Device:R
- added DI1: Diode_PESD5V0U2BT-Q, Package_TO_SOT_SMD:SOT-23, symbol Personal_Projects:Diode_PESD5V0U2BT-Q
- added FPC1: FPC_0545481072, Personal_Project:FPC_0545481072, symbol Personal_Projects:FPC_0545481072
- added FPC2: FPC_0545482072, Personal_Project:FPC_0545482072, symbol Personal_Projects:FPC_0545482072
- added J4: I2C1_Headers, Connector_PinHeader_2.54mm:PinHeader_2x03_P2.54mm_Horizontal, symbol Connector_Generic:Conn_02x03_Odd_Even
- added J5: UART1_HDR, Connector_PinHeader_2.54mm:PinHeader_2x03_P2.54mm_Horizontal, symbol Connector_Generic:Conn_02x03_Odd_Even
- added J6: I/O_HDR, symbol Connector_Generic:Conn_02x08_Odd_Even
- added R10, R3: 10k, Resistor_SMD:R_0805_2012Metric, symbol Device:R
- J24: value Debug_Pins -> SWDB
Connections:
- net GND: now also DI1.3 (CC), FPC1.1, FPC1.10, FPC1.11 (MP1), FPC1.12 (MP2), FPC1.3, FPC1.5, FPC1.6, FPC1.8, FPC2.1, FPC2.10, FPC2.11, FPC2.12, FPC2.14, FPC2.15, FPC2.17, FPC2.18, FPC2.20, FPC2.21 (MP1), FPC2.22 (MP2), FPC2.3, FPC2.4, FPC2.6, FPC2.7, FPC2.9, J4.2 (Pin_2), J4.3 (Pin_3), J4.4 (Pin_4), J4.6 (Pin_6), J5.1 (Pin_1), J5.2 (Pin_2), J5.4 (Pin_4), J5.5 (Pin_5), J5.6 (Pin_6), J6.10 (Pin_10), J6.12 (Pin_12), J6.14 (Pin_14), J6.16 (Pin_16), J6.2 (Pin_2), J6.4 (Pin_4), J6.6 (Pin_6), J6.8 (Pin_8)
- net at R5.2: now also J5.3 (Pin_3)
- net PA13_SWDIO renamed SWDIO
- net PA14_SWCLK renamed SWCLK
- net PA6_SPI1_MISO renamed UART1_TX/RX
- net PB3_SWO renamed SWO
- net PB5 renamed USR_BTN
- new net +3.3V: R10.1, R3.1
- new net I2C_SCL_HDR: DI1.2 (K2), J4.5 (Pin_5), R10.2
- new net I2C_SDA_HDR: DI1.1 (K1), J4.1 (Pin_1), R3.2
- new net I/O_HDR0: J6.1 (Pin_1)
- new net I/O_HDR1: J6.3 (Pin_3)
- new net I/O_HDR2: J6.5 (Pin_5)
- new net I/O_HDR3: J6.7 (Pin_7)
- new net I/O_HDR4: J6.9 (Pin_9)
- new net I/O_HDR5: J6.11 (Pin_11)
- new net I/O_HDR6: J6.13 (Pin_13)
- new net I/O_HDR7: J6.15 (Pin_15)
- new net QSPI_CLK: FPC2.2
- new net QSPI_CS0: FPC2.5
- new net QSPI_IO0: FPC2.8
- new net QSPI_IO1: FPC2.13
- new net QSPI_IO2: FPC2.16
- new net QSPI_IO3: FPC2.19
- new net SPI_CLK: FPC1.7
- new net SPI_CS: FPC1.9
- new net SPI_MISO: FPC1.4
- new net SPI_MOSI: FPC1.2
Other:
- note added: "Place ESD close to the header"
- note removed: "2.4 GHz band antenna"
- note removed: "Chip Select pin on general pin header"
- note removed: "Footprint: 0402"
- moved on the sheet: C21, J18, J24, U2

Commit message: Update
Parts:
- J4, J5: footprint Connector_PinHeader_2.54mm:PinHeader_2x03_P2.54mm_Horizontal -> Personal_Project:PinHeader_2x03_P2.54mm_Horizontal_Court
- J6: footprint (none) -> Connector_PinHeader_2.54mm:PinHeader_2x08_P2.54mm_Horizontal
Changed lines of the file:
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@@
 			)
 		)
-		(property "Footprint" "Connector_PinHeader_2.54mm:PinHeader_2x03_P2.54mm_Horizontal"
+		(property "Footprint" "Personal_Project:PinHeader_2x03_P2.54mm_Horizontal_Court"
 			(at 233.68 123.19 0)
 			(effects
@@
 			)
 		)
-		(property "Footprint" "Connector_PinHeader_2.54mm:PinHeader_2x03_P2.54mm_Horizontal"
+		(property "Footprint" "Personal_Project:PinHeader_2x03_P2.54mm_Horizontal_Court"
 			(at 81.28 118.11 0)
 			(effects
@@
 			)
 		)
-		(property "Footprint" ""
+		(property "Footprint" "Connector_PinHeader_2.54mm:PinHeader_2x08_P2.54mm_Horizontal"
 			(at 214.63 48.26 0)
 			(effects

Commit message: Update
Parts:
- removed FPC2: FPC_0545482072, Personal_Project:FPC_0545482072, symbol Personal_Projects:FPC_0545482072
- removed J18: User Button Jumper, Connector_PinHeader_2.54mm:PinHeader_1x02_P2.54mm_Vertical, symbol Connector_Generic:Conn_01x02
- removed J6: I/O_HDR, Connector_PinHeader_2.54mm:PinHeader_2x08_P2.54mm_Horizontal, symbol Connector_Generic:Conn_02x08_Odd_Even
- added J1: I/O_HDR, Connector_PinHeader_2.54mm:PinHeader_2x05_P2.54mm_Horizontal, symbol Connector_Generic:Conn_02x05_Odd_Even
Connections:
- net +3.3V: now also J1.1 (Pin_1)
- net GND: now also J1.3 (Pin_3), J1.5 (Pin_5), J1.7 (Pin_7), J1.9 (Pin_9)
- net I/O_HDR0: now also J1.2 (Pin_2)
- net I/O_HDR1: now also J1.4 (Pin_4)
- net I/O_HDR2: now also J1.6 (Pin_6)
- net I/O_HDR3: now also J1.8 (Pin_8)
- net I/O_HDR4: now also J1.10 (Pin_10)
- net USR_BTN: now also C21.2, U2.1, U2.2
Other:
- note removed: "Decide onn user button location ---------------"
- company: (none) -> Peter Hancak
- title: (none) -> STM32WB55RGVx Bleutooth Board
- moved on the sheet: C21, FPC1, J24, U2

Commit message: Update
Parts:
- removed FPC1: FPC_0545481072, Personal_Project:FPC_0545481072, symbol Personal_Projects:FPC_0545481072
- added FPC1: FPC_10051922-1010ELF, Personal_Project:FPC_10051922_1010, symbol Personal_Projects:FPC_10051922-1010ELF
Connections:
- net GND: now also FPC1.1, FPC1.10, FPC1.11 (MP1), FPC1.12 (MP2), FPC1.3, FPC1.5, FPC1.6, FPC1.8
- net SPI_CLK: now also FPC1.7
- net SPI_CS: now also FPC1.9
- net SPI_MISO: now also FPC1.4
- net SPI_MOSI: now also FPC1.2
Changed lines of the file:
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@@
-	)
-	(symbol
-		(lib_id "Personal_Projects:FPC_0545481072")
-		(at 53.34 41.91 0)
-		(unit 1)
-		(exclude_from_sim no)
-		(in_bom yes)
-		(on_board yes)
-		(dnp no)
-		(property "Reference" "FPC1"
-			(at 63.246 27.94 0)
-			(effects
-				(font
-					(size 1.27 1.27)
-				)
-				(justify right)
-			)
-		)
-		(property "Value" "FPC_0545481072"
-			(at 75.184 30.48 0)
-			(effects
-				(font
-					(size 1.27 1.27)
-				)
-				(justify right)
-			)
-		)
-		(property "Footprint" "Personal_Project:FPC_0545481072"
-			(at 74.93 136.83 0)
-			(effects
-				(font
-					(size 1.27 1.27)
-				)
-				(justify left top)
-				(hide yes)
-			)
-		)
-		(property "Datasheet" "https://www.molex.com/en-us/products/part-detail-pdf/545481072?display=pdf"
-			(at 74.93 236.83 0)
-			(effects
-				(font
-					(size 1.27 1.27)
-				)
-				(justify left top)
-				(hide yes)
-			)
-		)
-		(property "Description" "0.50mm Pitch Easy-On FFC/FPC Connector, 1.20mm Height, Right-Angle, Surface Mount, ZIF, Bottom Contact Style, 10 Circuits, Gold (Au) Plating"
-			(at 53.34 72.39 0)
-			(effects
-				(font
-					(size 1.27 1.27)
-				)
-				(hide yes)
-			)
-		)
-		(property "Height" "1.3"
-			(at 74.93 436.83 0)
-			(effects
-				(font
-					(size 1.27 1.27)
-				)
-				(justify left top)
-				(hide yes)
-			)
-		)
-		(property "Arrow Part Number" "0545481072"
-			(at 74.93 536.83 0)
-			(effects
-				(font
-					(size 1.27 1.27)
-				)
-				(justify left top)
-				(hide yes)
-			)
-		)
-		(property "Arrow Price/Stock" ""
-			(at 74.93 636.83 0)
-			(effects
-				(font
-					(size 1.27 1.27)
-				)
-				(justify left top)
-				(hide yes)
-			)
-		)
-		(property "Manufacturer_Name" "Molex"
-			(at 74.93 736.83 0)
-			(effects
-				(font
-					(size 1.27 1.27)
-				)
-				(justify left top)
-				(hide yes)
-			)
-		)
-		(property "Manufacturer_Part_Number" "0545481072"
-			(at 74.93 836.83 0)
-			(effects
-				(font
-					(size 1.27 1.27)
-				)
-				(justify left top)
-				(hide yes)
-			)
-		)
-		(pin "4"
-		)
-		(pin "7"
-		)
-		(pin "6"
-		)
-		(pin "5"
-		)
-		(pin "2"
-		)
-		(pin "8"
-		)
-		(pin "3"
-		)
-		(pin "10"
-		)
-		(pin "12"
-		)
-		(pin "11"
-		)
-		(pin "9"
-		)
-		(pin "1"
-		)
-		(instances
-			(project "Bluetooth_Board"
-				(path "/05989bb3-969e-4aaa-b344-5f0e2d5af968/abc98c8d-e19e-4e25-aa44-7b8f1ef72b8d"
-					(reference "FPC1")
-					(unit 1)
-				)
-			)
-		)
 	)
 	(symbol
@@
 					(unit 1)
 				)
+			)
+		)
+	)
+	(symbol
+		(lib_id "Personal_Projects:FPC_10051922-1010ELF")
+		(at 53.34 41.91 0)
+		(unit 1)
+		(exclude_from_sim no)
+		(in_bom yes)
+		(on_board yes)
+		(dnp no)
+		(property "Reference" "FPC1"
+			(at 64.77 25.654 0)
+			(effects
+				(font
+					(size 1.524 1.524)
+				)
+				(justify right)
+			)
+		)
+		(property "Value" "FPC_10051922-1010ELF"
+			(at 87.63 28.448 0)
+			(effects
+				(font
+					(size 1.524 1.524)
+				)
+				(justify right)
+			)
+		)
+		(property "Footprint" "Personal_Project:FPC_10051922_1010"
+			(at 53.34 88.9 0)
+			(effects
+				(font
+					(size 1.27 1.27)
+					(italic yes)
+				)
+				(hide yes)
+			)
+		)
+		(property "Datasheet" "10051922-1010ELF"
+			(at 53.34 85.09 0)
+			(effects
+				(font
+					(size 1.27 1.27)
+					(italic yes)
+				)
+				(hide yes)
+			)
+		)
+		(property "Description" ""
+			(at 66.04 41.91 0)
+			(effects
+				(font
+					(size 1.27 1.27)
+				)
+				(hide yes)
+			)
+		)
+		(pin "6"
+		)
+		(pin "9"
+		)
+		(pin "4"
+		)
+		(pin "7"
+		)
+		(pin "2"
+		)
+		(pin "5"
+		)
+		(pin "3"
+		)
+		(pin "8"
+		)
+		(pin "12"
+		)
+		(pin "10"
+		)
+		(pin "1"
+		)
+		(pin "11"
+		)
+		(instances
+			(project "Bluetooth_Board"
+				(path "/05989bb3-969e-4aaa-b344-5f0e2d5af968/abc98c8d-e19e-4e25-aa44-7b8f1ef72b8d"
+					(reference "FPC1")
+					(unit 1)
+				)
