File: Interfaces.kicad_sch (KiCad schematic)
At the start: 11 parts, among them J1 I/O_HDR, J24 SWDB, J4 I2C1_Headers, J5 UART1_HDR

Commit message: JLCPCB Check
Parts:
- added DI2, DI3: Diode_PESD5V0U2BT-Q, Package_TO_SOT_SMD:SOT-23, symbol Personal_Projects:Diode_PESD5V0U2BT-Q
- added FPC2: FPC_10051922-1010ELF, Personal_Project:FPC_10051922_1010, symbol Personal_Projects:FPC_10051922-1010ELF
- added H5, H6, H7, H8: MountingHole_Pad, MountingHole:MountingHole_3.2mm_M3_Pad, symbol Mechanical:MountingHole_Pad
- added J12: I/O_HDR, Connector_PinHeader_2.54mm:PinHeader_2x07_P2.54mm_Horizontal, symbol Connector_Generic:Conn_02x07_Odd_Even
- added J2: UART1_HDR, Personal_Projects:PinHeader_2x03_P2.54mm_Horizontal_Court, symbol Connector_Generic:Conn_02x03_Odd_Even
- added J8: I2C2_Headers, Personal_Project:PinHeader_2x03_P2.54mm_Horizontal_Court, symbol Connector_Generic:Conn_02x03_Odd_Even
- added J9: I2C1_Headers, Personal_Projects:PinHeader_2x03_P2.54mm_Horizontal_Court, symbol Connector_Generic:Conn_02x03_Odd_Even
- added R15: 33R, Resistor_SMD:R_0603_1608Metric, symbol Device:R
- added R21, R22: 10k, Resistor_SMD:R_0805_2012Metric, symbol Device:R
- added SHLD1: RFShield_OnePiece, Personal_Projects:RFSHIELD_MS353-30F, symbol Device:RFShield_OnePiece
- U2: value ~ -> (none)
Connections:
- net +3.3V: now also R21.1, R22.1
- net GND: now also DI2.3 (CC), DI3.3 (CC), FPC2.1, FPC2.10, FPC2.11 (MP1), FPC2.12 (MP2), FPC2.3, FPC2.5, FPC2.6, FPC2.8, H5.1, H6.1, H7.1, H8.1, J12.1 (Pin_1), J12.5 (Pin_5), J12.9 (Pin_9), J2.1 (Pin_1), J2.2 (Pin_2), J2.4 (Pin_4), J2.5 (Pin_5), J2.6 (Pin_6), J8.2 (Pin_2), J8.3 (Pin_3), J8.4 (Pin_4), J8.6 (Pin_6), J9.2 (Pin_2), J9.3 (Pin_3), J9.4 (Pin_4), J9.6 (Pin_6), SHLD1.1 (Shield)
- net I/O_HDR0: now also J12.2 (Pin_2)
- net I/O_HDR1: now also J12.4 (Pin_4)
- net I/O_HDR2: now also J12.6 (Pin_6)
- net I/O_HDR3: now also J12.8 (Pin_8)
- net I/O_HDR4: now also J12.10 (Pin_10)
- net SPI_CLK: now also FPC2.7
- net SPI_CS: now also FPC2.9
- net SPI_MISO: now also FPC2.4
- net SPI_MOSI: now also FPC2.2
- net UART1_TX/RX: now also R15.1
- new net: J2.3 (Pin_3), R15.2
- new net I2C_SCL_HDR_0: DI2.2 (K2), J9.5 (Pin_5), R22.2
- new net I2C_SCL_HDR_1: DI3.2 (K2), J8.5 (Pin_5)
- new net I2C_SDA_HDR_0: DI2.1 (K1), J9.1 (Pin_1), R21.2
- new net I2C_SDA_HDR_1: DI3.1 (K1), J8.1 (Pin_1)
- new net I/O_HDR10: J12.3 (Pin_3)
- new net I/O_HDR5: J12.12 (Pin_12)
- new net I/O_HDR6: J12.14 (Pin_14)
- new net I/O_HDR7: J12.13 (Pin_13)
- new net I/O_HDR8: J12.11 (Pin_11)
- new net I/O_HDR9: J12.7 (Pin_7)
Other:
- note added: "Alt: MS353-30C"
