File: STM32WB55CGU6.kicad_sch (KiCad schematic)
At the start: 25 parts, among them IC2 STM32WB55CGU6, J11 BOOT0_Jumper, J9 Coin Battery Jumper, Y1 ABM3B-32.000MHZ-8-R30-B1U-T

Commit message: Update
Parts:
- added C20: 47u, Capacitor_SMD:C_0805_2012Metric, symbol Device:C
Connections:
- net +3.3V: now also C20.1
- net GND: now also C20.2
- net PA10 renamed PA10_I2C1_SDA
- net PA2_LPUART1_TX renamed PA2_QUADSPI_BK1_NCS
- net PA3_LPUART1_RX renamed PA3_QUADSPI_CLK
- net PA6_SPI1_MISO renamed PA6_QUADSPI_BK1_IO3
- net PA7_SPI1_MOSI renamed PA7_QUADSPI_BK1_IO2
- net PA9 renamed PA9_I2C1_SCL
- net PB4 renamed PB4_SPI1_MISO
- net PB5 renamed PB5_SPI1_MOSI
- net PB7_USART1_RX renamed PB7
- net PB8_I2C1_SCL renamed PB8_QUADSPI_BK1_IO1
- net PB9_I2C1_SDA renamed PB9_QUADSPI_BK1_IO0
Other:
- company: (none) -> Peter Hancak
- title: (none) -> Bluetooth_STM32WB55_Board
- moved on the sheet: BH2, C1, C10, C11, C13, C14, C15, C16, C17, C18, C3, C4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

Commit message: Update
Parts:
- removed C15: 1u, Capacitor_SMD:C_0805_2012Metric, symbol Device:C
- removed C18: 100n, Capacitor_SMD:C_0805_2012Metric, symbol Device:C
- removed C20: 47u, Capacitor_SMD:C_0805_2012Metric, symbol Device:C
- removed FB2: BLM21PG601SN1D_0805, Capacitor_SMD:C_0805_2012Metric, symbol Device:FerriteBead

Commit message: Update
Parts:
- removed C17: 1uF, Capacitor_SMD:C_0805_2012Metric, symbol Device:C
- removed U1: ~, Personal_Project:Button_KMR231GLFS, symbol Personal_Projects:Button_KMR231GLFS
- L3: footprint Inductor_SMD:L_0402_1005Metric_Pad0.77x0.64mm_HandSolder -> Inductor_SMD:L_0805_2012Metric_Pad1.05x1.20mm_HandSolder

Commit message: Update
Parts:
- removed BH2: Battery_Holder_1060TR, Personal_Project:Battery_Holder_1060TR, symbol Personal_Projects:Battery_Holder_1060TR
- removed J9: Coin Battery Jumper, Connector_PinHeader_2.54mm:PinHeader_1x03_P2.54mm_Vertical, symbol Connector_Generic:Conn_01x03
- added C17: 100n, Capacitor_SMD:C_0805_2012Metric, symbol Device:C
- added MEM1: MX35LF2G24AD-Z4I, Package_DFN_QFN:WDFN-8-1EP_8x6mm_P1.27mm_EP6x4.8mm, symbol Personal_Projects:NAND_MX35LF2G24AD-Z4I
- added R1, R11, R12, R2, R9: 33R, Resistor_SMD:R_0805_2012Metric, symbol Device:R
Connections:
- net VBAT is gone; now on net +3.3V: C14.1, IC2.1 (VBAT)
- net +3.3V: now also C17.1, MEM1.8 (VCC)
- net GND: now also C17.2, MEM1.4 (GND), MEM1.9 (GND)
- net PA2_QUADSPI_BK1_NCS: now also MEM1.1 (CS#)
- net PA3_QUADSPI_CLK: now also R9.1
- net PA6_QUADSPI_BK1_IO3: now also R2.1
- net PA7_QUADSPI_BK1_IO2: now also R12.1
- net PB8_QUADSPI_BK1_IO1: now also R1.2
- net PB9_QUADSPI_BK1_IO0: now also R11.1
- net at IC2.2 (PC14-OSC32_IN): now also R4.1; no longer R4.2
- net at OS1.3 (OUTPUT): now also R4.2; no longer R4.1
- new net: MEM1.5 (SI/SIO0), R11.2
- new net: MEM1.7 (HOLD#/SIO3), R2.2
- new net: MEM1.3 (WP#/SIO2), R12.2
- new net: MEM1.2 (SO/SIO1), R1.1
- new net: MEM1.6 (SCLK), R9.2
- no-connect marks 5 -> 4
Other:
- note removed: "120ohm at 100MHz"
- note removed: "EP is optional adhesive zone"
- title: Bluetooth_STM32WB55_Board -> STM32WB55RGVx Bleutooth Board
- moved on the sheet: C14, R4

Commit message: Update
Parts:
- removed Y1: ABM3B-32.000MHZ-8-R30-B1U-T, Personal_Project:XTAL_ABM3B-32.000MHZ-10-R30-B1U-T, symbol Personal_Projects:ABM3B-32.000MHZ-10-R30-B1U-T
- added C23: 1n, Capacitor_SMD:C_0805_2012Metric, symbol Device:C
- added C28: 100n, Capacitor_SMD:C_0805_2012Metric, symbol Device:C
- added OS2: Oscillator_ATX-11-F-32.000MHZ-F05-T, Personal_Project:Oscillator_ECSTXO32CSMV320ANTR, symbol Personal_Projects:Oscillator_ECS-TXO-32CSMV-320-AN-TR
Connections:
- net +3.3V: now also C28.2, OS2.4 (VDD)
- net GND: now also C28.1, OS2.1 (GND_1), OS2.2 (GND_2)
- net OSC_IN: now also C23.1
- net OSC_OUT: no longer names the net of IC2.24 (OSC_OUT)
- new net OSC_OUTPUT: C23.2, OS2.3 (OUTPUT)
- no-connect marks 4 -> 5
Other:
- note added: "Clipped Sine Wave Oscillator - Series C eliminates DC component - MCU acciepots clock above zero so the clock signal gets biased (increased) inside the MCU."
- note removed: "Load Capacitors are inside the MCU Set RCC_HSECR register"
