File: STM32WB55CGU6.kicad_sch (KiCad schematic)
At the start: 27 parts, among them IC2 STM32WB55CGU6, J11 BOOT0_Jumper

Commit message: JLCPCB Check
Parts:
- removed C16: 10n, Capacitor_SMD:C_0805_2012Metric, symbol Device:C
- removed OS1: Oscillator_ECS-327MVATX-3-CN-TR, Personal_Project:Oscillator_ECS327MVATX3CNTR, symbol Personal_Projects:Oscillator_ECS-327MVATX-3-CN-TR
- removed R4: 10R, Resistor_SMD:R_0805_2012Metric, symbol Device:R
- added C25: 100n_CC0402KRX7R7BB104, Capacitor_SMD:C_0603_1608Metric, symbol Device:C
- added C29, C32: 10n, Capacitor_SMD:C_0603_1608Metric, symbol Device:C
- added C30: 47p_CC0402JRNPO9BN470, Capacitor_SMD:C_0603_1608Metric, symbol Device:C
- added C31: 10p, Capacitor_SMD:C_0603_1608Metric, symbol Device:C
- added C35: 1.2p_FGJM1555C1H1R2WB01D, Capacitor_SMD:C_0603_1608Metric, symbol Device:C
- added C71: 220n, Capacitor_SMD:C_0603_1608Metric, symbol Device:C
- added FB5: Murata_BLM21AG102SZ1D_1400R@1GHz, Capacitor_SMD:C_0805_2012Metric, symbol Device:FerriteBead
- added IC1: STM32WL55CCU6, Personal_Projects:STM32WL55CCU6_QFN50P700X700X65-49N-D, symbol Personal_Components:STM32WL55CCU6
- added J13, J14: BOOT0_J, Connector_PinHeader_2.54mm:PinHeader_2x03_P2.54mm_Vertical, symbol Connector_Generic:Conn_02x03_Odd_Even
- added OS3, OS5: Oscillator_ECS-327MVATX-3-CN-TR, Crystal:Crystal_SMD_3225-4Pin_3.2x2.5mm, symbol Personal_Projects:Oscillator_ECS-327MVATX-3-CN-TR
- added OS4: Oscillator_HCI 8132S-32.000MN33DTL, Crystal:Crystal_SMD_3225-4Pin_3.2x2.5mm, symbol Personal_Projects:Oscillator_ECS-TXO-32CSMV-320-AN-TR
- added R13: 220R, Resistor_SMD:R_0603_1608Metric, symbol Device:R
- added R14, R6: 10R, Resistor_SMD:R_0603_1608Metric, symbol Device:R
- added R32, R33: 10k, Resistor_SMD:R_0805_2012Metric, symbol Device:R
- added U16, U17: (no value), Personal_Project:Button_SKSCLCE010, symbol Personal_Projects:BTN_SKSCLCE010
Connections:
- net +3.3V: now also U16.3, U16.4, U17.3, U17.4
- net BOOT0: now also IC1.19 (PH3-BOOT0), J13.2 (Pin_2), J13.4 (Pin_4), J13.6 (Pin_6), J14.2 (Pin_2), J14.4 (Pin_4), J14.6 (Pin_6)
- net GND: now also C25.2, C29.1, C30.2, C32.1, C35.2, C71.1, OS3.2 (GND), OS4.1 (GND_1), OS4.2 (GND_2), OS5.2 (GND), R32.1, R33.1
- net NRST: now also IC1.18 (NRST)
- net PA15: now also IC1.43 (PA15)
- net PB6_USART1_TX: now also IC1.4 (PB6)
- net PC14-OSC32_IN: now reaches IC2.2 (PC14-OSC32_IN)
- net PC14-OSC32_IN: now also IC1.26 (OSC_IN), R14.1, R6.1
- net PC15-OSC32_OUT: now reaches IC2.3 (PC15-OSC32_OUT)
- net PC15-OSC32_OUT: now also IC1.27 (OSC_OUT)
- new net: C71.2, FB5.2, OS4.4 (VDD)
- new net: OS3.3 (OUTPUT), R6.2
- new net: OS5.3 (OUTPUT), R14.2
- new net +3.3VLOAD: C29.2, C32.2, OS3.1 (TRI-STATE), OS3.4 (VDD), OS5.1 (TRI-STATE), OS5.4 (VDD)
- new net BOOT0J: J13.5 (Pin_5), J14.5 (Pin_5), R32.2, R33.2, U16.1, U16.2, U17.1, U17.2
- new net BOOT0_EXTCTR: J13.3 (Pin_3), J14.3 (Pin_3)
- new net BOOT0_GPIO: J13.1 (Pin_1), J14.1 (Pin_1)
- new net OSC_IN_1: C31.1, R13.2
- new net OSC_IN_2: OS4.3 (OUTPUT), R13.1
- new net PA0_USART2_CTS: IC1.7 (PA0)
- new net PA10_SPI2_MOSI: IC1.33 (PA10)
- new net PA11_DEBUG_RF-NRESET: IC1.34 (PA11)
- new net PA12_DEBUG_RF-BUSY: IC1.35 (PA12)
- new net PA13_DEBUG_JTMS-SWDIO: IC1.36 (PA13)
- new net PA14_DEBUG_JTCK-SWCLK: IC1.42 (PA14)
- new net PA1_USART2_RTS: IC1.8 (PA1)
- new net PA2_USART2_TX: IC1.9 (PA2)
- new net PA3_USART2_RX: IC1.10 (PA3)
- new net PA4: IC1.12 (PA4)
- new net PA5_SPI2_MISO: IC1.13 (PA5)
- new net PA6: IC1.14 (PA6)
- new net PA7_DEBUG_SUBGHZSPIMOSIOUT: IC1.15 (PA7)
- new net PA8_RCC_MCO: IC1.16 (PA8)
- new net PA9_SPI2_SCK: IC1.17 (PA9)
- new net PB0_VDD_TCXO+: C25.1, C30.1, C35.1, FB5.1
- new net PB12_SPI2_NSS: IC1.32 (PB12)
- new net PB2_DEBUG_RF-SMPSRDY: IC1.31 (PB2)
- new net PB3_DEBUG_JTDO-SWO: IC1.1 (PB3)
- new net PB4_DEBUG_RF-LDORDY: IC1.2 (PB4)
- new net PB5: IC1.3 (PB5)
- new net PB7_I2C1_SDA: IC1.5 (PB7)
- new net PB8_I2C1_SCL: IC1.6 (PB8)
- new net PC13: IC1.38 (PC13)
- new net PH0-OSC_IN: C31.2, IC1.39 (PC14-OSC32_IN)
- new net PH1-OSC_OUT: IC1.40 (PC15-OSC32_OUT)
- no-connect marks 5 -> 4
Other:
- note added: "Clipped Sine Wave Oscillator - Series C eliminates DC component - MCU acciepots clock above zero so the clock signal gets biased (increased) inside the MCU. Alt: ATX-11-F-32.000MHZ-F05-T"
- note added: "EN set by SMPS_TPS62740DSSR"
- note added: "Internal pullup resistor allows active output if pin 1 is NC"
- note added: "OSC32OUT Can be used as GPIO"
- note added: "Place near the TCXO"
- note added: "Reference design: BLM15HG102SN1"
- note removed: "NRST has internal pull-up resistor -When button not pushed NRST is HIGH -Pushing the button causes current to flow and pulls NRST low"
- note removed: "The external capacitor on NRST must be placed as close as possible to the device."
- moved on the sheet: J11
