File: RF.kicad_sch (KiCad schematic)
At the start: 18 parts, among them J1 USB_C_Receptacle_USB2.0_16P, J3 SMA PCB END LAUNCH JACK ROUND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, U3 USBLC6-2SC6

Commit message: Update
Parts:
- removed C22: 100p, Capacitor_SMD:C_0805_2012Metric, symbol Device:C
- removed C23: 100n, Capacitor_SMD:C_0805_2012Metric, symbol Device:C
- removed C24: 10u, Capacitor_SMD:C_0805_2012Metric, symbol Device:C
- removed C25: 47u, Capacitor_SMD:C_0805_2012Metric, symbol Device:C
- removed J1: USB_C_Receptacle_USB2.0_16P, Connector_USB:USB_C_Receptacle_HRO_TYPE-C-31-M-12, symbol Connector:USB_C_Receptacle_USB2.0_16P
- removed R1, R2: 5k1, Resistor_SMD:R_0805_2012Metric, symbol Device:R
- removed U3: USBLC6-2SC6, Package_TO_SOT_SMD:SOT-23-6, symbol Power_Protection:USBLC6-2SC6
- removed Z1: Diode_BZX84C6V2-7-F, Personal_Project:Diode_BZX84C6V2_SOT96P240X110-3N, symbol Personal_Projects:Diode_BZX84C6V2-7-F
- added C26, C28: 100n, Capacitor_SMD:C_0805_2012Metric, symbol Device:C
- added C27: 4u7, Capacitor_SMD:C_0805_2012Metric, symbol Device:C
- added FB1: Part # MI0805K601R-10, Capacitor_SMD:C_0805_2012Metric, symbol Device:FerriteBead
- added J7: USB_C_Receptacle_USB2.0_16P, Connector_USB:USB_C_Receptacle_HRO_TYPE-C-31-M-12, symbol Connector:USB_C_Receptacle_USB2.0_16P
- added R7, R8: 5k1, Resistor_SMD:R_0805_2012Metric, symbol Device:R
- added U5: USBLC6-2SC6, Package_TO_SOT_SMD:SOT-23-6, symbol Power_Protection:USBLC6-2SC6
- added Z2: Diode_BZX84C6V2-7-F, Personal_Project:Diode_BZX84C6V2_SOT96P240X110-3N, symbol Personal_Projects:Diode_BZX84C6V2-7-F
Connections:
- net GND: now also C26.2, C27.2, C28.2, J7.A1 (GND), J7.A12 (GND), J7.B1 (GND), J7.B12 (GND), J7.S1 (SHIELD), R7.2, R8.2, U5.2 (GND), Z2.1 (A)
- net USB_D2+: now also J7.A6 (D+), J7.B6 (D+), U5.4 (I/O2)
- net USB_D2+_DI: now also U5.3 (I/O2)
- net USB_D2-: now also J7.A7 (D-), J7.B7 (D-), U5.6 (I/O1)
- net USB_D2-_DI: now also U5.1 (I/O1)
- net USB_VBUS+: now also C26.1, C27.1, C28.1, FB1.1, FB1.2, J7.A4 (VBUS), J7.A9 (VBUS), J7.B4 (VBUS), J7.B9 (VBUS), U5.5 (VBUS), Z2.3 (K)
- new net: J7.A5 (CC1), R7.1
- new net: J7.B5 (CC2), R8.1
Other:
- note added: "------Maybe add diode on the 5V power"
- note added: "600 Ohms @ 100 MHz"
- note added: "Matched Net Lengths [Tolerance = 2mm] Impedance Constraint [Min = 85.00 Max = 95.00 ]"

Commit message: Update
Connections:
- net USB_VBUS+: no longer C28.1, FB1.1, J7.A4 (VBUS), J7.A9 (VBUS), J7.B4 (VBUS), J7.B9 (VBUS), U5.5 (VBUS), Z2.3 (K)
- new net USB_VBUS_P+: C28.1, FB1.1, J7.A4 (VBUS), J7.A9 (VBUS), J7.B4 (VBUS), J7.B9 (VBUS), U5.5 (VBUS), Z2.3 (K)
Changed lines of the file:
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@@
+	)
+	(junction
+		(at 86.36 57.15)
+		(diameter 0)
+		(color 0 0 0 0)
 	)
 	(junction
@@
 	(wire
 		(pts
-			(xy 86.36 55.88) (xy 86.36 58.42)
+			(xy 86.36 55.88) (xy 86.36 57.15)
 		)
 		(stroke
@@
 		(pts
 			(xy 224.79 128.27) (xy 226.06 128.27)
+		)
+		(stroke
+			(width 0)
+			(type default)
+		)
+	)
+	(wire
+		(pts
+			(xy 86.36 57.15) (xy 86.36 58.42)
 		)
 		(stroke
@@
 		)
 	)
-	(label "USB_VBUS+"
+	(label "USB_VBUS_P+"
 		(at 196.85 100.33 0)
 		(fields_autoplaced yes)
@@
 					(unit 1)
 				)
+			)
+		)
+	)
+	(symbol
+		(lib_id "power:PWR_FLAG")
+		(at 86.36 57.15 90)
+		(unit 1)
+		(exclude_from_sim no)
+		(in_bom yes)
+		(on_board yes)
+		(dnp no)
+		(fields_autoplaced yes)
+		(property "Reference" "#FLG03"
+			(at 84.455 57.15 0)
+			(effects
+				(font
+					(size 1.27 1.27)
+				)
+				(hide yes)
+			)
+		)
+		(property "Value" "PWR_FLAG"
+			(at 81.28 57.15 0)
+			(effects
+				(font
+					(size 1.27 1.27)
+				)
+				(hide yes)
+			)
+		)
+		(property "Footprint" ""
+			(at 86.36 57.15 0)
+			(effects
+				(font
+					(size 1.27 1.27)
+				)
+				(hide yes)
+			)
+		)
+		(property "Datasheet" "~"
+			(at 86.36 57.15 0)
+			(effects
+				(font
+					(size 1.27 1.27)
+				)
+				(hide yes)
+			)
+		)
+		(property "Description" "Special symbol for telling ERC where power comes from"
+			(at 86.36 57.15 0)
+			(effects
+				(font
+					(size 1.27 1.27)
+				)
+				(hide yes)
+			)
+		)
+		(pin "1"
+		)
+		(instances
+			(project "Bluetooth_Board"
+				(path "/05989bb3-969e-4aaa-b344-5f0e2d5af968/1ac22050-21cc-40c3-9af0-4a5defc56765"
+					(reference "#FLG03")
+					(unit 1)
+				)

Commit message: Update
Connections:
- net USB_D2+: now also U5.6 (I/O1); no longer U5.4 (I/O2)
- net USB_D2-: now also U5.4 (I/O2); no longer U5.6 (I/O1)
- net USB_D2+_DI renamed USB_DI_D2-
- net USB_D2-_DI renamed USB_DI_D2+
Other:
- moved on the sheet: U5
Changed lines of the file:
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@@
 	)
 	(junction
-		(at 219.71 128.27)
-		(diameter 0)
-		(color 0 0 0 0)
-	)
-	(junction
 		(at 110.49 113.03)
 		(diameter 0)
@@
 	)
 	(junction
+		(at 219.71 128.27)
+		(diameter 0)
+		(color 0 0 0 0)
+	)
+	(junction
 		(at 233.68 161.29)
 		(diameter 0)
@@
 	(wire
 		(pts
-			(xy 177.8 153.67) (xy 177.8 128.27)
+			(xy 177.8 123.19) (xy 177.8 153.67)
 		)
 		(stroke
@@
 	(wire
 		(pts
+			(xy 173.99 125.73) (xy 180.34 125.73)
+		)
+		(stroke
+			(width 0)
+			(type default)
+		)
+	)
+	(wire
+		(pts
 			(xy 166.37 55.88) (xy 166.37 58.42)
 		)
@@
 	(wire
 		(pts
-			(xy 190.5 128.27) (xy 219.71 128.27)
+			(xy 190.5 123.19) (xy 194.31 123.19)
 		)
 		(stroke
@@
 	(wire
 		(pts
-			(xy 185.42 133.35) (xy 185.42 161.29)
+			(xy 185.42 130.81) (xy 185.42 161.29)
 		)
 		(stroke
@@
 	(wire
 		(pts
-			(xy 185.42 100.33) (xy 185.42 120.65)
+			(xy 185.42 100.33) (xy 185.42 118.11)
+		)
+		(stroke
+			(width 0)
+			(type default)
+		)
+	)
+	(wire
+		(pts
+			(xy 190.5 125.73) (xy 219.71 125.73)
 		)
 		(stroke
@@
 	(wire
 		(pts
+			(xy 180.34 123.19) (xy 177.8 123.19)
+		)
+		(stroke
+			(width 0)
+			(type default)
+		)
+	)
+	(wire
+		(pts
 			(xy 224.79 102.87) (xy 219.71 102.87)
 		)
@@
 	(wire
 		(pts
-			(xy 173.99 125.73) (xy 180.34 125.73)
+			(xy 194.31 123.19) (xy 194.31 128.27)
 		)
 		(stroke
@@
 	(wire
 		(pts
-			(xy 190.5 125.73) (xy 219.71 125.73)
-		)
-		(stroke
-			(width 0)
-			(type default)
-		)
-	)
-	(wire
-		(pts
 			(xy 153.67 100.33) (xy 153.67 102.87)
 		)
@@
 	(wire
 		(pts
-			(xy 67.31 172.72) (xy 58.42 172.72)
+			(xy 194.31 128.27) (xy 219.71 128.27)
 		)
 		(stroke
@@
 	(wire
 		(pts
-			(xy 110.49 100.33) (xy 110.49 102.87)
+			(xy 67.31 172.72) (xy 58.42 172.72)
 		)
 		(stroke
@@
 	(wire
 		(pts
-			(xy 110.49 100.33) (xy 124.46 100.33)
+			(xy 110.49 100.33) (xy 110.49 102.87)
 		)
 		(stroke
@@
 	(wire
 		(pts
-			(xy 177.8 128.27) (xy 180.34 128.27)
+			(xy 110.49 100.33) (xy 124.46 100.33)
 		)
 		(stroke
@@
 		)
 	)
-	(label "USB_D2+_DI"
+	(label "USB_DI_D2+"
 		(at 118.11 153.67 0)
 		(fields_autoplaced yes)
@@
 		)
 	)
-	(label "USB_D2-_DI"
+	(label "USB_DI_D2-"
 		(at 118.11 151.13 0)
 		(fields_autoplaced yes)
@@
 		)
 	)
-	(hierarchical_label "USB_D2+_DI"
+	(hierarchical_label "USB_DI_D2+"
 		(shape bidirectional)
 		(at 118.11 153.67 180)
@@
 		)
 	)
-	(hierarchical_label "USB_D2-_DI"
+	(hierarchical_label "USB_DI_D2-"
 		(shape bidirectional)
 		(at 118.11 151.13 180)
@@
 	(symbol
 		(lib_id "Power_Protection:USBLC6-2SC6")
-		(at 185.42 125.73 0)
+		(at 185.42 123.19 0)
 		(unit 1)
 		(exclude_from_sim no)
@@
 		(dnp no)
 		(property "Reference" "U5"
-			(at 186.182 118.364 0)
+			(at 186.182 115.824 0)
 			(effects
 				(font
@@
 		)
 		(property "Value" "USBLC6-2SC6"
-			(at 186.182 120.65 0)
+			(at 186.182 118.11 0)
 			(effects
 				(font
@@
 		)
 		(property "Footprint" "Package_TO_SOT_SMD:SOT-23-6"
-			(at 186.69 132.08 0)
+			(at 186.69 129.54 0)
 			(effects
 				(font
@@
 		)
 		(property "Datasheet" "https://www.st.com/resource/en/datasheet/usblc6-2.pdf"
-			(at 186.69 133.985 0)
+			(at 186.69 131.445 0)
 			(effects
 				(font
@@
 		)
 		(property "Description" "Very low capacitance ESD protection diode, 2 data-line, SOT-23-6"
-			(at 185.42 125.73 0)
+			(at 185.42 123.19 0)
 			(effects
 				(font

Commit message: Update
Connections:
- net USB_VBUS+ renamed VBUS+
- net USB_VBUS_P+ renamed VBUS_P+
Other:
- company: (none) -> Peter Hancak
- title: (none) -> STM32WB55RGVx Bleutooth Board
Changed lines of the file:
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@@
 	(generator_version "8.0")
 	(paper "USLetter")
+	(title_block
+		(title "STM32WB55RGVx Bleutooth Board")
+		(date "2024-11-22")
+		(rev "A")
+		(company "Peter Hancak")
+	)
 	(junction
 		(at 224.79 130.81)
@@
 		)
 	)
-	(label "USB_VBUS_P+"
+	(label "VBUS_P+"
 		(at 196.85 100.33 0)
 		(fields_autoplaced yes)
@@
 			)
 		)
-		(property "Value" "USB_VBUS+"
-			(at 93.472 94.488 0)
-			(effects
-				(font
+		(property "Value" "VBUS+"
+			(at 90.932 95.758 0)
+			(effects
+				(font

Commit message: Update
Parts:
- removed C26, C28: 100n, Capacitor_SMD:C_0805_2012Metric, symbol Device:C
- removed FB1: Part # MI0805K601R-10, Capacitor_SMD:C_0805_2012Metric, symbol Device:FerriteBead
Connections:
- net VBUS_P+ is gone; now on net VBUS+: J7.A4 (VBUS), J7.A9 (VBUS), J7.B4 (VBUS), J7.B9 (VBUS), U5.5 (VBUS), Z2.3 (K)
Other:
- note removed: "------Maybe add diode on the 5V power"
- note removed: "600 Ohms @ 100 MHz"

Commit message: Update
Parts:
- C19: value 0p8 GRM1555C1HR80BA01D -> 1p3 GRM1555C1HR80BA01D
- C2: value 0p3 GRM1555C1HR30WA01D -> 1p GRM1555C1HR30WA01D
- L1: value 2n7 LQG15HS2N7S02 -> 3n LQG15HS2N7S02
Other:
- note added: "STM32WB55CGU6 RF pin input impedance is 42+j19 Ω"
Changed lines of the file:
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@@
+		)
+	)
+	(text "STM32WB55CGU6 RF pin input impedance is 42+j19 Ω"
+		(exclude_from_sim no)
+		(at 173.228 79.756 0)
+		(effects
+			(font
+				(size 1 1)
+			)
 		)
 	)
@@
 			)
 		)
-		(property "Value" "0p3 GRM1555C1HR30WA01D"
+		(property "Value" "1p GRM1555C1HR30WA01D"
 			(at 140.716 68.326 90)
 			(effects
@@
 			)
 		)
-		(property "Value" "2n7 LQG15HS2N7S02"
+		(property "Value" "3n LQG15HS2N7S02"
 			(at 155.194 47.244 90)
 			(effects
@@
 			)
 		)
-		(property "Value" "0p8 GRM1555C1HR80BA01D"
+		(property "Value" "1p3 GRM1555C1HR80BA01D"
 			(at 170.434 68.58 90)
 			(effects

Commit message: Update
Parts:
- C19: value 1p3 GRM1555C1HR80BA01D -> 1p5 GRM1555C1HR80BA01D
- C2: value 1p GRM1555C1HR30WA01D -> 1p2 GRM1555C1HR30WA01D
- L1: value 3n LQG15HS2N7S02 -> 2n9 LQG15HS2N7S02
Changed lines of the file:
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@@
 			)
 		)
-		(property "Value" "1p GRM1555C1HR30WA01D"
+		(property "Value" "1p2 GRM1555C1HR30WA01D"
 			(at 140.716 68.326 90)
 			(effects
@@
 				)
 				(justify left)
+				(hide yes)
 			)
 		)
@@
 			)
 		)
-		(property "Value" "3n LQG15HS2N7S02"
+		(property "Value" "2n9 LQG15HS2N7S02"
 			(at 155.194 47.244 90)
 			(effects
@@
 			)
 		)
-		(property "Value" "1p3 GRM1555C1HR80BA01D"
+		(property "Value" "1p5 GRM1555C1HR80BA01D"
 			(at 170.434 68.58 90)
 			(effects
